File: eagle/oresatt-batteries.brd (EAGLE design)
At the start: 94 x 93.5 mm, 62 parts, among them IC1 74AHC1G08DBV, U1 TCAN330, U2 STM32F042K6, X1 16MHz

Commit message: Cleaned up schematic, moved STC sense resistor to proper place.
Connections:
- net N$3 renamed ANDDRIVE
- new net C_SENSE: R3.2, R6.2, U$13.P$1, U$13.P$2, U$13.P$3, U$5.6
- net GND: no longer R3.2, R6.2, U$13.P$1, U$13.P$2, U$13.P$3, U$5.6
Changed lines of the file:
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@@
 <contactref element="C4" pad="2"/>
 <contactref element="C5" pad="2"/>
-<contactref element="R3" pad="1"/>
 <contactref element="R4" pad="1"/>
 <contactref element="U$5" pad="5"/>
@@
 <contactref element="C13" pad="2"/>
 <contactref element="R12" pad="1"/>
-<contactref element="U$13" pad="P$1"/>
-<contactref element="U$13" pad="P$2"/>
-<contactref element="U$13" pad="P$3"/>
 <contactref element="DEBUG_DNP" pad="15"/>
 <contactref element="DEBUG_DNP" pad="16"/>
 <contactref element="U$21" pad="V-"/>
 <contactref element="IC1" pad="3"/>
-<contactref element="R6" pad="2"/>
-<contactref element="R3" pad="2"/>
-<contactref element="U$5" pad="6"/>
 <contactref element="C14" pad="2"/>
+<contactref element="R3" pad="1"/>
 <wire x1="21.85" y1="80.08" x2="20.85" y2="81.93" width="0" layer="19" extent="1-1"/>
-<wire x1="21.795" y1="75.42" x2="21.85" y2="80.08" width="0" layer="19" extent="1-1"/>
-<wire x1="22.415" y1="75.42" x2="21.795" y2="75.42" width="0" layer="19" extent="1-1"/>
+<wire x1="22.415" y1="75.42" x2="21.85" y2="80.08" width="0" layer="19" extent="1-1"/>
 <wire x1="17.325" y1="78.375" x2="21.85" y2="80.08" width="0" layer="19" extent="1-1"/>
 <wire x1="15.675" y1="79.625" x2="17.325" y2="78.375" width="0" layer="19" extent="1-1"/>
@@
 <wire x1="14.2" y1="66.75" x2="13.35" y2="70" width="0" layer="19" extent="1-1"/>
 <wire x1="11.65" y1="76" x2="13.35" y2="73" width="0" layer="19" extent="1-1"/>
-<wire x1="9.35" y1="76" x2="11.65" y2="76" width="0" layer="19" extent="1-1"/>
-<wire x1="7.65" y1="73" x2="9.35" y2="76" width="0" layer="19" extent="1-1"/>
+<wire x1="7.65" y1="73" x2="11.65" y2="76" width="0" layer="19" extent="1-1"/>
 <wire x1="27.175" y1="72.2" x2="22.415" y2="75.42" width="0" layer="19" extent="1-1"/>
 <wire x1="24.85" y1="68.5" x2="27.175" y2="72.2" width="0" layer="19" extent="1-1"/>
@@
 <wire x1="24.85" y1="53" x2="20.85" y2="52.5" width="0" layer="19" extent="1-1"/>
 <wire x1="27.65" y1="53" x2="24.85" y2="53" width="0" layer="19" extent="1-1"/>
-<wire x1="29.35" y1="53" x2="27.65" y2="53" width="0" layer="19" extent="1-1"/>
-<wire x1="29.35" y1="57" x2="29.35" y2="53" width="0" layer="19" extent="1-1"/>
+<wire x1="29.35" y1="57" x2="27.65" y2="53" width="0" layer="19" extent="1-1"/>
 <wire x1="4.25" y1="52.5" x2="14.65" y2="52.5" width="0" layer="19" extent="1-1"/>
 <wire x1="15.15" y1="41.5" x2="14.65" y2="52.5" width="0" layer="19" extent="1-1"/>
@@
 <wire x1="10.39" y1="-13.73" x2="32.5" y2="21" width="0" layer="19" extent="16-16"/>
 <wire x1="10.39" y1="-16.27" x2="10.39" y2="-13.73" width="0" layer="19" extent="1-1"/>
-<wire x1="-3.175" y1="-3.435" x2="10.39" y2="-13.73" width="0" layer="19" extent="1-1"/>
-<wire x1="-3.825" y1="-3.435" x2="-3.175" y2="-3.435" width="0" layer="19" extent="1-1"/>
-<wire x1="-4.475" y1="-3.435" x2="-3.825" y2="-3.435" width="0" layer="19" extent="1-1"/>
-<wire x1="-26.95" y1="-39.09" x2="-4.475" y2="-3.435" width="0" layer="19" extent="1-1"/>
+<wire x1="-26.95" y1="-39.09" x2="10.39" y2="-16.27" width="0" layer="19" extent="1-1"/>
 <wire x1="-28.55" y1="-49.4" x2="-26.95" y2="-39.09" width="0" layer="19" extent="1-1"/>
 </signal>
@@
 <contactref element="U2" pad="18"/>
 </signal>
-<signal name="N$3">
+<signal name="ANDDRIVE">
 <contactref element="U$14" pad="P$4"/>
 <contactref element="IC1" pad="4"/>
@@
 <wire x1="-2.525" y1="-3.435" x2="26.66" y2="76.825" width="0" layer="19" extent="1-1"/>
 </signal>
+<signal name="C_SENSE">
+<contactref element="R6" pad="2"/>
+<contactref element="R3" pad="2"/>
+<contactref element="U$13" pad="P$1"/>
+<contactref element="U$13" pad="P$2"/>
+<contactref element="U$13" pad="P$3"/>
+<contactref element="U$5" pad="6"/>
+<wire x1="9.35" y1="76" x2="21.795" y2="75.42" width="0" layer="19" extent="1-1"/>
+<wire x1="29.35" y1="53" x2="21.795" y2="75.42" width="0" layer="19" extent="1-1"/>
+<wire x1="-3.175" y1="-3.435" x2="29.35" y2="53" width="0" layer="19" extent="1-1"/>
+<wire x1="-3.825" y1="-3.435" x2="-3.175" y2="-3.435" width="0" layer="19" extent="1-1"/>
+<wire x1="-4.475" y1="-3.435" x2="-3.825" y2="-3.435" width="0" layer="19" extent="1-1"/>
+</signal>
 </signals>

Commit message: Schematic Cleanup, added labels and isolated chips visually
Connections:
- net VBATT+: now also R10.2
Changed lines of the file:
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@@
 <contactref element="U$3" pad="POS"/>
 <contactref element="R7" pad="2"/>
+<contactref element="R10" pad="2"/>
 <wire x1="23.7" y1="80.08" x2="23.7" y2="79.58" width="0" layer="19" extent="1-1"/>
 <wire x1="23.7" y1="80.58" x2="23.7" y2="80.08" width="0" layer="19" extent="1-1"/>
@@
 <wire x1="21.25" y1="59.7" x2="23.15" y2="61" width="0" layer="19" extent="1-1"/>
 <wire x1="20.85" y1="56.5" x2="21.25" y2="59.7" width="0" layer="19" extent="1-1"/>
+<wire x1="24.85" y1="57" x2="20.85" y2="56.5" width="0" layer="19" extent="1-1"/>
 <wire x1="23.15" y1="53" x2="20.85" y2="56.5" width="0" layer="19" extent="1-1"/>
-<wire x1="29.35" y1="64.5" x2="23.15" y2="64.5" width="0" layer="19" extent="1-1"/>
-<wire x1="29.35" y1="60.5" x2="29.35" y2="64.5" width="0" layer="19" extent="1-1"/>
+<wire x1="29.35" y1="60.5" x2="24.85" y2="57" width="0" layer="19" extent="1-1"/>
+<wire x1="29.35" y1="64.5" x2="29.35" y2="60.5" width="0" layer="19" extent="1-1"/>
 <wire x1="16.45" y1="49.6" x2="23.15" y2="53" width="0" layer="19" extent="1-1"/>
 <wire x1="12.75" y1="62.1" x2="21.25" y2="59.7" width="0" layer="19" extent="1-1"/>
