File: eagle/oresat-batteries-v1.1.sch (EAGLE design)
At the start: 102 parts, among them IC1 74AHC1G08DBV, J1 2MM-RA-1X8, Q1 CSD16340Q3, Q2 CSD16340Q3, Q3 TPN4R712MD, Q4 TPN4R712MD, Q5 TPN4R712MD, Q6 TPN4R712MD, Q7 CSD16340Q3, U1 LM3761, U10 LTC4412, U11 MAX17055, U12 LTC4412, U13 LTC4412, U14 STM32F042K6, U15 TCAN330, U2 MC74HC1G04DFT1GOSCT, U3 BQ2970, U4 LTC4411, U5 LTC4411, U6 LTC4411, U7 LTC4411, U8 MC74HC1G04DFT1GOSCT, U9 LTC4412, X1 16MHz

Commit message: Cosmeticas.
Other:
- note added: "- Still need to select a thermister. - Still need to select fuses."
- note removed: "- Still need to select a thermister. - Still need to select fuses. - Still need diodes and connection to MCU from CHG/DCHG_CTL - Change test points from U$ to TP* - Change mostfets to Q$"
- moved on the sheet: B1, C1, C10, C11, C12, C13, C14, C15, C2, C3, C4, C5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
