File: eagle/oresat-batteries.sch (EAGLE design)
At the start: 106 parts, among them IC1 74AHC1G08DBV, J1 J-SAMTEC-TFM-120-X1-XXX-D-RA, J7 1.27MM-SWD-CONNECTOR, Q1 CSD16340Q3, Q10 TPN4R712MD, Q11 TPN4R712MD, Q12 TPN4R712MD, Q2 CSD16340Q3, Q3 TPN4R712MD, Q4 TPN4R712MD, Q5 TPN4R712MD, Q6 TPN4R712MD, Q8 TPN4R712MD, Q9 TPN4R712MD, U1 TPS63070, U10 LTC4412, U11 MAX17055, U12 LTC4412, U13 LTC4412, U2 TCAN330, U3 BQ2970, U4 LTC4411, U5 LTC4411, U6 STM32F042K6, U7 LTC4411, U8 LTC4411, U9 LTC4412, X1 16MHZ-2.5x2mm

Commit message: New 2S2P battery boards, based on 18650 cells along with a BQ28400 battery IC.
Parts:
- removed C11, C16: 20p, rcl_custom:C-EU0402-B-NOSILK
- removed C14: 22u, oresat-rcl:C-EU0603-B-NOSILK
- removed C17, C22: 100n, rcl_custom:C-EU0402-B-NOSILK
- removed C18, C25: 22u, oresat-rcl:C-EU0805-B-NOSILK
- removed D1, D2, D3: GREEN, SparkFun-LED:LED-GREEN0603
- removed F2: 2016L500DR, F-LITTELFUSE-2016L-SERIES-PTC:F-LITTELFUSE-2016L-SERIES-PTC
- removed H1, H2, H3, H4: STAND-OFFTIGHT, SparkFun-Hardware:STAND-OFFTIGHT
- removed IC1: 74AHC1G08DBV, 74xx-little-us:74AHC1G08DBV
- removed J1: J-SAMTEC-TFM-120-X1-XXX-D-RA, J-Samtec-TFM-120-X1-XXX-D-RA:J-SAMTEC-TFM-120-X1-XXX-D-RA
- removed J5: (no value), SparkFun-Connectors:6_PIN_SERIAL_TARGETSILK
- removed J7: 1.27MM-SWD-CONNECTOR, J-CNC-3220-10-0100-00-ARM-SWD-port:1.27MM-SWD-CONNECTOR
- removed JP8: (no value), pinhead:PINHD-1X2
- removed L3: 1.5 uH, L-Coilcraft-XFL4020:L-COILCRAFT-XFL4020
- removed Q10, Q11, Q12, Q6, Q8, Q9: TPN4R712MD, tpn4r712md-pmosfet:TPN4R712MD
- removed R18: NP, rcl_custom:R-US_0402-B-NOSILK
- removed R19, R21, R26, R28, R29: 10k, rcl:R-US_R0603
- removed R20: 4.19, oresat-batteries:RES_HEATER
- removed R22, R23, R24, R25: 470k, rcl:R-US_R0603
- removed R27: 3.3k, rcl:R-US_R0402
- removed R3: 2.7k, rcl_custom:R-US_0402-B-NOSILK
- removed TP10, TP11, TP12, TP13, TP14, TP16, TP17, TP20, TP6, TP7, TP8, TP9: TP, oresat-batteries:TP
- removed TP15, TP4, TP5: TEST-POINT, Tova:TEST-POINT
- removed U10, U12, U13, U9: LTC4412, ltc4412:LTC4412
- removed U11: MAX17055, max17055:MAX17055
- removed U2: TCAN330, TCAN330:TCAN330
- removed U3: BQ2970, oresat-batteries:BQ2970
- removed U4, U5, U7, U8: LTC4411, ltc4411:LTC4411
- removed U6: STM32F042K6, STM32F042K:STM32F042K6
- removed X1: 16MHZ-2.5x2mm, low-gain-radio:CRYSTAL-WITH-GND
- added B2, B3, B4: B-18650-LI-BATTERY, B-18650-Li-battery:B-18650-LI-BATTERY
- added J6: J-SAMTEC-TFM-120-X1-XXX-D-RA, J-Samtec-TFM-120-X1-XXX-D-RA:J-SAMTEC-TFM-120-X1-XXX-D-RA
- added TR1: 10k, oresat-rcl:R-US_0603-B-NOSILK
- B1: value 2AHBATT -> B-18650-LI-BATTERY; device oresat-batteries:2AHBATT -> B-18650-Li-battery:B-18650-LI-BATTERY
- C1: value .1u -> 1u; device rcl:C-EUC0603 -> oresat-rcl:C-EU0603-B-NOSILK
- C10, C7: value .1u -> 100n; device rcl:C-EUC0603 -> oresat-rcl:C-EU0402-B-NOSILK
- C2: value .47u -> 100n; device rcl:C-EUC0603 -> oresat-rcl:C-EU0402-B-NOSILK
- C3, C5, C9: device rcl_custom:C-EU0402-B-NOSILK -> oresat-rcl:C-EU0402-B-NOSILK; DIS Digi-Key -> (none); DPN 1276-1001-1-ND -> (none); MFR Samsung -> (none); MPN CL05B104KO5NNNC -> (none)
- C4: value 10u -> 100n; device oresat-rcl:C-EU0603-B-NOSILK -> oresat-rcl:C-EU0402-B-NOSILK; DIS Digi-Key -> (none); DPN 1276-1001-1-ND -> (none); MFR Samsung -> (none); MPN CL05B104KO5NNNC -> (none)
- C6: value 10u -> 1u; device oresat-rcl:C-EU0805-B-NOSILK -> oresat-rcl:C-EU0603-B-NOSILK
- C8: value 10u -> 100n; device oresat-rcl:C-EU0805-B-NOSILK -> oresat-rcl:C-EU0402-B-NOSILK
- F1: DIS Digi-Key -> (none); DPN 2016L200PRCT-ND -> (none); MFR Littelfuse -> (none); MPN 2016L200PR -> (none)
- Q1, Q2: value CSD16340Q3 -> MOSFET-PCH-SOT23-6; device oresat-batteries:CSD16340Q3 -> Q-MOSFET-PCH-SOT23-6:MOSFET-PCH-SOT23-6
- Q3, Q4, Q5: device tpn4r712md-pmosfet:TPN4R712MD -> Q-Toshiba-TPN4R712MD-MOSFET-P-CH-Power:TPN4R712MD
- R1: value 2.7k -> 10m; device rcl_custom:R-US_0402-B-NOSILK -> oresat-rcl:R-US_M2012; DIS Digi-Key -> (none); DPN 1276-4275-1-ND -> (none); MFR Samsung -> (none); MPN RC1005F6653CS -> (none)
- R10: value 470k -> 100; device rcl_custom:R-US_0402-B-NOSILK -> oresat-rcl:R-US_1206-B; DIS Digi-Key -> (none); DPN 1276-4275-1-ND -> (none); MFR Samsung -> (none); MPN RC1005F6653CS -> (none)
- R11: value 4.7k -> 3M; device rcl:R-US_R0603 -> oresat-rcl:R-US_0603-B-NOSILK
- R12: value 100k -> 3M; device rcl_custom:R-US_0402-B-NOSILK -> oresat-rcl:R-US_0603-B-NOSILK; DIS Digi-Key -> (none); DPN 1276-4275-1-ND -> (none); MFR Samsung -> (none); MPN RC1005F6653CS -> (none)
- R13: value 10k -> 5.1k; device rcl:R-US_R0603 -> oresat-rcl:R-US_0603-B-NOSILK
- R14: value 2.2k -> 5.1k; device rcl:R-US_R0603 -> oresat-rcl:R-US_0603-B-NOSILK
- R15: value 10k -> 1M; device rcl_custom:R-US_0402-B-NOSILK -> oresat-rcl:R-US_0603-B-NOSILK; DIS Digi-Key -> (none); DPN 1276-4275-1-ND -> (none); MFR Samsung -> (none); MPN RC1005F6653CS -> (none)
- R16: value NP -> 5.1k; device rcl_custom:R-US_0402-B-NOSILK -> oresat-rcl:R-US_0603-B-NOSILK; DIS Digi-Key -> (none); DPN 1276-4275-1-ND -> (none); MFR Samsung -> (none); MPN RC1005F6653CS -> (none)
- R17: value 10k -> 221; device rcl_custom:R-US_0402-B-NOSILK -> oresat-rcl:R-US_M2012; DIS Digi-Key -> (none); DPN 1276-4275-1-ND -> (none); MFR Samsung -> (none); MPN RC1005F6653CS -> (none)
- R2: value 2.7k -> 1k; device rcl_custom:R-US_0402-B-NOSILK -> oresat-rcl:R-US_0603-B-NOSILK; DIS Digi-Key -> (none); DPN 1276-4275-1-ND -> (none); MFR Samsung -> (none); MPN RC1005F6653CS -> (none)
- R4: value .01-.05 -> 0? 1k?; device rcl:R-US_R2512 -> oresat-rcl:R-US_0603-B-NOSILK
- R5: value 2.2k -> 100; device rcl:R-US_R0603 -> oresat-rcl:R-US_0402-B-NOSILK
- R6: value 330 -> 100; device rcl:R-US_R0603 -> oresat-rcl:R-US_0402-B-NOSILK
- R7: value 10k -> 1k; device rcl_custom:R-US_0402-B-NOSILK -> oresat-rcl:R-US_0402-B-NOSILK; DIS Digi-Key -> (none); DPN 1276-4275-1-ND -> (none); MFR Samsung -> (none); MPN RC1005F6653CS -> (none)
- R8: value 4.7k -> 1k; device rcl:R-US_R0603 -> oresat-rcl:R-US_0402-B-NOSILK
- R9: value DNP/0 -> 100; device rcl:R-US_R0603 -> oresat-rcl:R-US_1206-B
- U$1: value MMBT3904-TP -> ORESAT-CARD-V0.5; device mmbt3904-tp:MMBT3904-TP -> oresat-card:ORESAT-CARD-V0.5
- U1: value TPS63070 -> BQ28400; device ic-pwr-tps63070x:TPS63070X -> U-TI-BQ28400-Li-battery-monitor:BQ28400; DIS Digi-Key -> (none); DPN 296-44874-1-ND -> (none); MFR TI -> (none); MPN TPS63070 -> (none)
Connections:
- removed net !SYSSHD: IC1A.I0, J1.7, J1.8, R14.2, TP8.P$1
- removed net .3556: Q4.D, Q9.D, U10.SENSE, U13.VIN
- removed net 3.3V: C14.1, C17.2, C18.1, C22.2, C25.1, C3.2, C9.2, J7.VTREF, R10.2, R11.2, R13.2, R16.2, R2.2, R22.1, R23.1, R24.1, R25.1, R8.2, TP1.1, U1.VOUT, U2.VCC, U6.VDD, U6.VDDA, U6.VDDIO2
- removed net 4411MB: U7.OUT, U8.IN
- removed net 4411_MT: U4.OUT, U5.IN
- removed net ALERT: R13.1, R9.2, TP17.P$1, U11.ALRT
- removed net ANDDRIVE: IC1A.O, Q1.G
- removed net BATT-: B1.V-, IC1P.GND, Q1.S, TP20.P$1, U3.VSS
- removed net BETSHUT: Q1.D, Q2.D
- removed net BGDOUT: IC1A.I1, TP10.P$1, U3.DOUT
- removed net BOOT: R17.2, TP15.1, U6.PB8-BOOT0
- removed net BQBAT: C1.1, R6.1, TP6.P$1, U3.BAT
- removed net BQCOUT: Q2.G, TP9.P$1, U3.COUT
- removed net BQVMIN: R5.1, U3.V-
- removed net CAN_H: J1.3, J1.4, U2.CANH
- removed net CAN_L: J1.1, J1.2, U2.CANL
- removed net CAN_RX: U2.RXD, U6.PA11
- removed net CAN_SHDN: U2.SHDN, U6.PA10
- removed net CAN_SILENT: U2.S, U6.PA9
- removed net CAN_TX: U2.TXD, U6.PA12
- removed net CHARGE-STAT-U4-U5: R25.2, U4.STAT, U5.STAT, U6.PA5
- removed net CHARGE-STAT-U7-U8: R24.2, U6.PA4, U7.STAT, U8.STAT
- removed net CHARGE_ENABLE: R29.2, TP11.P$1, U4.CTL, U5.CTL, U6.PB1, U7.CTL, U8.CTL
- removed net CRYSTALIN: C16.1, U6.PF0-OSC_IN, X1.1
- removed net CRYSTALOUT: C11.1, U6.PF1-OSC_OUT, X1.2
- removed net C_SENSE: Q2.S, R21.1, R4.2, R5.2, TP13.P$1, U11.CSP
- removed net DISCHARGE-STAT-U10-U13: R23.2, U12.STAT, U6.PA7, U9.STAT
- removed net DISCHARGE-STAT-U9-U12: R22.2, U10.STAT, U13.STAT, U6.PA6
- removed net DISCHARGE_ENABLE: R26.1, TP14.P$1, U10.CTL, U12.CTL, U13.CTL, U6.PB3, U9.CTL
- removed net HEAT: R27.1, U6.PB0
- removed net HEAT_FET_CTL: Q12.G, R28.1, U$1.C
- removed net INFUSE: F1.P$1, U4.IN, U7.IN
- removed net MAX_IO: R9.1, U6.PA1
- removed net N$1: D3.A, R3.1
- removed net N$2: Q3.S, Q8.S
- removed net N$270: D1.A, R1.1
- removed net N$271: D2.A, R2.1
- removed net N$3: Q10.S, Q5.S
- removed net N$4: Q11.S, Q4.S
- removed net N$406: J5.VCC, JP8.2
- removed net N$436: Q10.G, Q5.G, U12.GATE
- removed net N$437: Q10.D, Q3.D, U12.VIN, U9.SENSE
- removed net N$438: Q3.G, Q8.G, U9.GATE
- removed net N$439: Q6.G, Q9.G, U13.GATE
- removed net N$441: Q11.G, Q4.G, U10.GATE
- removed net N$5: Q6.S, Q9.S
- removed net N$6: Q12.D, R20.1
- removed net N$7: R27.2, U$1.B
- removed net NRESET: J7.!RESET, U6.NRST
- removed net OUTFUSE: F2.P$2, Q5.D, Q6.D, U12.SENSE, U13.SENSE
- removed net PA0: R3.2, U6.PA0
- removed net PA2/USART2_TX: J5.TXO, U6.PA2
- removed net PA3/USART2_RX: J5.RXI, U6.PA3
- removed net REG: C2.1, U11.REG
- removed net SCL: R11.1, TP7.P$1, U11.SCL, U6.PB6
- removed net SDA: R8.1, TP16.P$1, U11.SDA, U6.PB7
- removed net SPARE10: J1.35, J1.36
- removed net SPARE11: J1.37, J1.38
- removed net SPARE12: J1.39, J1.40
- removed net SPARE8: J1.31, J1.32
- removed net SPARE9: J1.33, J1.34
- removed net SWCLK: J7.SWDCLK/TCK, U6.PA14-SWCLK
- removed net SWDIO: J7.SWDIO/TMS, U6.PA13-SWDIO
- removed net TEMPSENSE: R19.1, R21.2, U11.AIN
- removed net THRM: R19.2, U11.THRM
- removed net TPS-EN1: R18.2, R7.1, TP5.1, U1.EN, U1.PS/SYNC
- removed net TPS-FB1: R10.1, R12.2, U1.FB
- removed net TPS-FB3: TP3.1, U1.FB2
- removed net TPS-L3: L3.1, U1.L1
- removed net TPS-L4: L3.2, U1.L2
- removed net TPS-PG1: R16.1, TP2.1, U1.PG
- removed net TPS-VAUX1: C5.1, U1.VAUX
- removed net TPS-VSEL1: R15.2, TP4.1, U1.VSEL
- removed net V_BATT: B1.V+, C10.1, C7.1, IC1P.VCC, Q11.D, Q12.S, Q8.D, R14.1, R28.2, R6.2, TP12.P$1, U10.VIN, U11.BATT, U5.OUT, U8.OUT, U9.VIN
- new net !CB_EN: TP1.1, U1.!CB_EN
- new net !PRES: R2.1, U1.!PRES
- new net !SHUTDOWN: J6.39, J6.40
- new net BQ-SCLK: TP3.1, U1.SMBC
- new net BQ-SDA: TP2.1, U1.SMBD
- new net CAN1_H: J6.33, J6.34
- new net CAN1_L: J6.35, J6.36
- new net CAN2_H: J6.21, J6.22
- new net CAN2_L: J6.23, J6.24
- new net CHG: R13.2, U1.CHG
- new net DSG: R14.2, U1.DSG
- new net FUSE: R4.1, U1.FUSE
- new net GNDA: B3.NEG, B4.NEG, C1.2, C2.2, C3.2, C4.2, C6.2, C7.2, C8.2, R1.2, R2.2, R4.2, R6.1, R9.1, TR1.1, U1.VSS
- new net N$10: Q1.D, R9.2
- new net N$11: Q2.D, R10.2
- new net N$13: Q3.D, Q4.D, R17.2
- new net N$14: Q3.G, R11.2, R13.1
- new net N$15: Q4.G, R12.2, R14.1
- new net N$18: Q5.G, R15.2, R16.1
- new net N$20: Q5.D, R17.1
- new net N$21: C10.1, C9.2
- new net OPD_PWR: J6.19, J6.20
- new net OPD_SCL: J6.17, J6.18
- new net OPD_SDA: J6.15, J6.16
- new net PACK: C9.1, F1.P$1, Q3.S, Q5.S, R11.1, R15.1, U1.PACK
- new net RBI: C2.1, U1.RBI
- new net REG27: C1.1, U1.REG27
- new net SRN: C3.1, C5.1, R5.2, U1.SRN
- new net SRP: C4.1, C5.2, R6.2, U1.SRP
- new net TS1: TR1.2, U1.TS1
- new net V1S: B1.NEG, B2.NEG, B3.POS, B4.POS, Q1.S, R10.1, R8.2
- new net V2S: B1.POS, B2.POS, C10.2, C6.1, Q2.S, Q4.S, R12.1, R7.2, U1.BAT
- new net VC1: C8.1, Q2.G, R7.1, U1.VC1
- new net VC2: C7.1, Q1.G, R8.1, U1.VC2
- new net ZVCHG: R16.2, U1.ZVCHG
- net GND: now also J6.29, J6.30, J6.31, J6.32, J6.37, J6.38, R1.1, R5.1; no longer C1.2, C10.2, C11.2, C14.2, C16.2, C17.1, C18.2, C2.2, C22.1, C25.2, C3.1, C4.2, C5.2, C6.2, C7.2, C8.2, C9.1, D1.C, D2.C, D3.C, J1.10, J1.11, J1.12, J1.5, J1.6, J1.9, J5.GND, J7.GND, J7.GND@2, J7.GNDDET, R12.1, R15.1, R17.1, R18.1, R20.2, R26.2, R29.1, R4.1, U$1.E, U1.GND, U1.PGND, U10.GND, U11.CSN, U12.GND, U13.GND, U2.GND, U4.GND, U5.GND, U6.VSS, U7.GND, U8.GND, U9.GND, X1.SHIELD
- net SPARE1: now also J6.13, J6.14; no longer J1.17, J1.18
- net SPARE2: now also J6.11, J6.12; no longer J1.19, J1.20
- net SPARE3: now also J6.10, J6.9; no longer J1.21, J1.22
- net SPARE4: now also J6.7, J6.8; no longer J1.23, J1.24
- net SPARE5: now also J6.5, J6.6; no longer J1.25, J1.26
- net SPARE6: now also J6.3, J6.4; no longer J1.27, J1.28
- net SPARE7: now also J6.1, J6.2; no longer J1.29, J1.30
- net VBUS: now also J6.25, J6.26, J6.27, J6.28; no longer C4.1, C6.1, C8.1, F2.P$1, J1.13, J1.14, J1.15, J1.16, JP8.1, R1.2, R7.2, U1.VIN
Other:
- note added: "(49.5 88.769)"
- note added: "1206"
- note added: "2012"
- note added: "2012 1/2W"
- note added: "2A cont, 4A trip."
- note added: "OreSat Power Domain signals (See power sheet)"
- note added: "REPLACE WITH 0 OHM FOR FLIGHT"
- note added: "thermistor"
- note removed: "-3.9V"
- note removed: "0805"
- note removed: "1.1"
- note removed: "10 pn 1.27mm ARM SWD connector"
- note removed: "2A cont, 4A trip"
- note removed: "3.36V Nom"
- note removed: "5A cont, 10A trip"
- note removed: "All caps are ceramic 10% X5R >= 16V Vwv unless marked"
- note removed: "All resistors 0402 +/- 1% unless marked"
- note removed: "CAN Transceiver"
- note removed: "Cell Protection"
- note removed: "Fuel Gauge"
- note removed: "Input current: - 4 x 250 mA = 1 A from solar - Inrush from batteries with higher voltage - External chargers (1C only)"
- note removed: "Iq = 10uA"
- note removed: "Iq = 4uA"
- note removed: "Low = Charge"
- note removed: "Low = Discharge"
- note removed: "Low = on"
- note removed: "Meant for FTDI TTL-232R-3V3 cable"
- note removed: "NRST pull-up built in"
- note removed: "OreSat Proto-Card"
- note removed: "Output curent: - < 100 mA in standby - < 2 A in 70 cm TX - < 5 A in S Band TX"
- note removed: "PCB TRACE HEATER"
- note removed: "Power VBUS from USB 5V (DEV ONLY)"
- note removed: "REPLACE with 0 ohm for flight?"
- note removed: "Thermister"
- note removed: "Vbus = (3.0, 3.6, 4.2) V"

Commit message: update schematic with s8209 and MAX17205 chips for battery protection and control
Parts:
- removed F1: 2016L200PR, F-LITTELFUSE-2016L-SERIES-PTC:F-LITTELFUSE-2016L-SERIES-PTC
- removed TR1: 10k, oresat-rcl:R-US_0603-B-NOSILK
- added C11, C16: 20p, rcl_custom:C-EU0402-B-NOSILK
- added C12: 22u, oresat-rcl:C-EU0805-B-NOSILK
- added C13, C15: 1n, oresat-rcl:C-USC0402
- added C14: .1u, oresat-rcl:C-USC0402
- added C17, C22: 100n, rcl_custom:C-EU0402-B-NOSILK
- added C18: 10n, rcl:C-USC0402K
- added C19, C21: 100n, rcl:C-USC0402K
- added D1, D2: GREEN, SparkFun-LED:LED-GREEN0603
- added D4: AMBER, SparkFun-LED:LED-GREEN0603
- added J1: J-SAMTEC-TFM-110-X1-XXX-D-RA, J-Samtec-TFM-110-X1-XXX-D-RA:J-SAMTEC-TFM-110-X1-XXX-D-RA
- added L2: 6.8u, L-ECS-MPI4040:L-ECS-MPI4040
- added Q6: PMV45EN, Tova:PMV45EN
- added R18, R26, R27, R28, R30, R35, R38: 10k, rcl_custom:R-US_0402-B-NOSILK
- added R19, R20, R21, R22, R23, R32, R34, R36, R37: NP, rcl_custom:R-US_0402-B-NOSILK
- added R24, R25: 100, rcl_custom:R-US_0402-B-NOSILK
- added R29: 100m, rcl:R-US_R1206
- added R3, R46, R49, R50: 4.7k, rcl:R-US_R0402
- added R31, R33: 0, rcl_custom:R-US_0402-B-NOSILK
- added R39: 10, oresat-rcl:R-US_0603-B
- added R40: .01, rcl:R-US_R0805
- added R41, R42: 10k, rcl:R-US_R0603
- added R43, R44: 10k, oresat-rcl:R-US_R0603
- added R47, R48, R51, R52: 1k, rcl:R-US_R0402
- added R53, R54: 470, rcl:R-US_R0402
- added R55: 100, rcl:R-US_R0603
- added TP10, TP11, TP12, TP13, TP14, TP15, TP16, TP17, TP18, TP19, TP20, TP4, TP5, TP6, TP8, TP9: TEST-POINT, Tova:TEST-POINT
- added U$3, U$4: S8209A, U-ABLIC-s8209A-BattProtection:S8209A
- added U2: TCAN330, TCAN330:TCAN330
- added U3: MAX7310ATE, U-Maxim-MAX7310-I2C-GPIO-expander:MAX7310
- added U4: MAX4211CETE, U-Maxim-MAX4211-power-monitor:MAX4211
- added U5: TPS62111RSA, U-TI-TPS6211x-SPS-buck:TPS6211X
- added U6: STM32F042K6, STM32F042K:STM32F042K6
- added U7: MCP1703A, v-reg:XC63FPM
- added X1: 16MHZ-2.5x2mm, low-gain-radio:CRYSTAL-WITH-GND
- C1: value 1u -> 100n; device oresat-rcl:C-EU0603-B-NOSILK -> rcl_custom:C-EU0402-B-NOSILK; DIS (none) -> Digi-Key; DPN (none) -> 1276-1001-1-ND; MFR (none) -> Samsung; MPN (none) -> CL05B104KO5NNNC
- C10, C4, C5: value 100n -> 1u; device oresat-rcl:C-EU0402-B-NOSILK -> oresat-rcl:C-EU0603-B-NOSILK; DIS (none) -> Digi-Key; DPN (none) -> 1276-1001-1-ND; MFR (none) -> Samsung; MPN (none) -> CL05B104KO5NNNC
- C2: value 100n -> NP; device oresat-rcl:C-EU0402-B-NOSILK -> rcl_custom:C-EU0402-B-NOSILK; DIS (none) -> Digi-Key; DPN (none) -> 1276-1001-1-ND; MFR (none) -> Samsung; MPN (none) -> CL05B104KO5NNNC
- C3, C9: device oresat-rcl:C-EU0402-B-NOSILK -> rcl_custom:C-EU0402-B-NOSILK; DIS (none) -> Digi-Key; DPN (none) -> 1276-1001-1-ND; MFR (none) -> Samsung; MPN (none) -> CL05B104KO5NNNC
- C6: value 1u -> TBD; device oresat-rcl:C-EU0603-B-NOSILK -> rcl_custom:C-EU0402-B-NOSILK; DIS (none) -> Digi-Key; DPN (none) -> 1276-1001-1-ND; MFR (none) -> Samsung; MPN (none) -> CL05B104KO5NNNC
- C7: value 100n -> 10u; device oresat-rcl:C-EU0402-B-NOSILK -> oresat-rcl:C-EU0805-B-NOSILK
- C8: value 100n -> TBD; device oresat-rcl:C-EU0402-B-NOSILK -> rcl_custom:C-EU0402-B-NOSILK; DIS (none) -> Digi-Key; DPN (none) -> 1276-1001-1-ND; MFR (none) -> Samsung; MPN (none) -> CL05B104KO5NNNC
- Q1: value MOSFET-PCH-SOT23-6 -> DMP2240UDM; device Q-MOSFET-PCH-SOT23-6:MOSFET-PCH-SOT23-6 -> Q-MOSFET-PCH-dual-SOT23-6:MOSFET-PCH-SOT23-6; MFR (none) -> Diodes Inc; MPN (none) -> DMP2240UDM
- Q2: device Q-MOSFET-PCH-SOT23-6:MOSFET-PCH-SOT23-6 -> Q-MOSFET-PCH-dual-SOT23-6:MOSFET-PCH-SOT23-6
- Q3, Q4: value TPN4R712MD -> MOSFET-PCH-SOT23-6; device Q-Toshiba-TPN4R712MD-MOSFET-P-CH-Power:TPN4R712MD -> Q-MOSFET-PCH-SOT23-6:MOSFET-PCH-SOT23-6; MFR (none) -> Diodes Inc; MPN (none) -> DMP3050LVT-7
- Q5: value TPN4R712MD -> PMV45EN; device Q-Toshiba-TPN4R712MD-MOSFET-P-CH-Power:TPN4R712MD -> Tova:PMV45EN
- R1: value 10m -> 2.7k; device oresat-rcl:R-US_M2012 -> rcl_custom:R-US_0402-B-NOSILK; DIS (none) -> Digi-Key; DPN (none) -> 1276-4275-1-ND; MFR (none) -> Samsung; MPN (none) -> RC1005F6653CS
- R10, R9: value 100 -> NP; device oresat-rcl:R-US_1206-B -> rcl_custom:R-US_0402-B-NOSILK; DIS (none) -> Digi-Key; DPN (none) -> 1276-4275-1-ND; MFR (none) -> Samsung; MPN (none) -> RC1005F6653CS
- R11: value 3M -> NP; device oresat-rcl:R-US_0603-B-NOSILK -> rcl_custom:R-US_0402-B-NOSILK; DIS (none) -> Digi-Key; DPN (none) -> 1276-4275-1-ND; MFR (none) -> Samsung; MPN (none) -> RC1005F6653CS
- R12: value 3M -> 2.7k; device oresat-rcl:R-US_0603-B-NOSILK -> rcl_custom:R-US_0402-B-NOSILK; DIS (none) -> Digi-Key; DPN (none) -> 1276-4275-1-ND; MFR (none) -> Samsung; MPN (none) -> RC1005F6653CS
- R13, R14: value 5.1k -> NP; device oresat-rcl:R-US_0603-B-NOSILK -> rcl_custom:R-US_0402-B-NOSILK; DIS (none) -> Digi-Key; DPN (none) -> 1276-4275-1-ND; MFR (none) -> Samsung; MPN (none) -> RC1005F6653CS
- R15: value 1M -> 10k; device oresat-rcl:R-US_0603-B-NOSILK -> rcl_custom:R-US_0402-B-NOSILK; DIS (none) -> Digi-Key; DPN (none) -> 1276-4275-1-ND; MFR (none) -> Samsung; MPN (none) -> RC1005F6653CS
- R16: value 5.1k -> 10k; device oresat-rcl:R-US_0603-B-NOSILK -> rcl_custom:R-US_0402-B-NOSILK; DIS (none) -> Digi-Key; DPN (none) -> 1276-4275-1-ND; MFR (none) -> Samsung; MPN (none) -> RC1005F6653CS
- R17: value 221 -> 10k; device oresat-rcl:R-US_M2012 -> rcl_custom:R-US_0402-B-NOSILK; DIS (none) -> Digi-Key; DPN (none) -> 1276-4275-1-ND; MFR (none) -> Samsung; MPN (none) -> RC1005F6653CS
- R2: value 1k -> 2.7k; device oresat-rcl:R-US_0603-B-NOSILK -> rcl_custom:R-US_0402-B-NOSILK; DIS (none) -> Digi-Key; DPN (none) -> 1276-4275-1-ND; MFR (none) -> Samsung; MPN (none) -> RC1005F6653CS
- R4: value 0? 1k? -> 100; device oresat-rcl:R-US_0603-B-NOSILK -> rcl_custom:R-US_0402-B-NOSILK; DIS (none) -> Digi-Key; DPN (none) -> 1276-4275-1-ND; MFR (none) -> Samsung; MPN (none) -> RC1005F6653CS
- R5, R6: value 100 -> NP; device oresat-rcl:R-US_0402-B-NOSILK -> rcl_custom:R-US_0402-B-NOSILK; DIS (none) -> Digi-Key; DPN (none) -> 1276-4275-1-ND; MFR (none) -> Samsung; MPN (none) -> RC1005F6653CS
- R7: value 1k -> 10k; device oresat-rcl:R-US_0402-B-NOSILK -> rcl_custom:R-US_0402-B-NOSILK; DIS (none) -> Digi-Key; DPN (none) -> 1276-4275-1-ND; MFR (none) -> Samsung; MPN (none) -> RC1005F6653CS
- R8: value 1k -> NP; device oresat-rcl:R-US_0402-B-NOSILK -> rcl_custom:R-US_0402-B-NOSILK; DIS (none) -> Digi-Key; DPN (none) -> 1276-4275-1-ND; MFR (none) -> Samsung; MPN (none) -> RC1005F6653CS
- U$1: value ORESAT-CARD-V0.5 -> ORESAT-CARD-V1.1-3XRF; device oresat-card:ORESAT-CARD-V0.5 -> oresat-cards:ORESAT-CARD-V1.1-3XRF
- U1: value BQ28400 -> MAX17205G; device U-TI-BQ28400-Li-battery-monitor:BQ28400 -> U-Maxim-MAX17205-Fuel_Gauge:MAX17205G+00E
Connections:
- net CAN2_H renamed N$525
- net CAN2_L renamed N$524
- net SPARE1 renamed N$528
- net SPARE2 renamed N$500
- net SPARE3 renamed N$503
- net SPARE5 renamed N$504
- net SPARE6 renamed N$519
- net SPARE7 renamed N$520
- removed net !CB_EN: TP1.1, U1.!CB_EN
- removed net !PRES: R2.1, U1.!PRES
- removed net BQ-SCLK: TP3.1, U1.SMBC
- removed net BQ-SDA: TP2.1, U1.SMBD
- removed net CHG: R13.2, U1.CHG
- removed net DSG: R14.2, U1.DSG
- removed net FUSE: R4.1, U1.FUSE
- removed net GNDA: B3.NEG, B4.NEG, C1.2, C2.2, C3.2, C4.2, C6.2, C7.2, C8.2, R1.2, R2.2, R4.2, R6.1, R9.1, TR1.1, U1.VSS
- removed net N$13: Q3.D, Q4.D, R17.2
- removed net N$18: Q5.G, R15.2, R16.1
- removed net N$20: Q5.D, R17.1
- removed net N$21: C10.1, C9.2
- removed net PACK: C9.1, F1.P$1, Q3.S, Q5.S, R11.1, R15.1, U1.PACK
- removed net RBI: C2.1, U1.RBI
- removed net REG27: C1.1, U1.REG27
- removed net SRN: C3.1, C5.1, R5.2, U1.SRN
- removed net SRP: C4.1, C5.2, R6.2, U1.SRP
- removed net TS1: TR1.2, U1.TS1
- removed net V2S: B1.POS, B2.POS, C10.2, C6.1, Q2.S, Q4.S, R12.1, R7.2, U1.BAT
- removed net VC1: C8.1, Q2.G, R7.1, U1.VC1
- removed net VC2: C7.1, Q1.G, R8.1, U1.VC2
- removed net ZVCHG: R16.2, U1.ZVCHG
- new net !FAULT: Q6.D, R38.1, TP8.1, U3.IO2
- new net 3.3V: C12.1, C17.2, C22.2, C3.2, C9.2, L2.2, R2.2, TP17.1, U2.VCC, U5.FB, U6.VDD, U6.VDDA, U6.VDDIO2
- new net AD0: R5.1, R6.2, R8.2, R9.1, U3.AD0
- new net AD1: R11.1, R13.2, R14.2, R19.1, U3.AD1
- new net AD2: R20.1, R21.2, R22.2, R23.1, U3.AD2
- new net AUX_!SHUTDOWN: J1.19, J1.20
- new net AUX_CAN1_H: J1.13, J1.14
- new net AUX_CAN1_L: J1.15, J1.16
- new net AUX_CAN2_H: J1.1, J1.2
- new net AUX_CAN2_L: J1.3, J1.4
- new net AUX_GND1: J1.17, J1.18
- new net AUX_GND2: J1.11, J1.12
- new net AUX_GND3: J1.10, J1.9
- new net AUX_VBUS1: J1.7, J1.8
- new net AUX_VBUS2: J1.5, J1.6
- new net BOOT: R17.2, TP15.1, U6.PB8-BOOT0
- new net CAN_RX: U2.RXD, U6.PA11
- new net CAN_SHDN: U2.SHDN, U6.PA10
- new net CAN_SILENT: U2.S, U6.PA9
- new net CAN_TX: U2.TXD, U6.PA12
- new net CB-RESET: R30.2, TP14.1, U3.IO1, U4.CIN2+
- new net CB_CTRL: Q3.G, Q6.G, R35.1, U4.COUT1, U4.COUT2, U4.LE
- new net CRYSTALIN: C16.1, U6.PF0-OSC_IN, X1.1
- new net CRYSTALOUT: C11.1, U6.PF1-OSC_OUT, X1.2
- new net MAX4211-3V3: C5.1, U4.VCC, U7.OUT
- new net N$1: R3.2, R46.2
- new net N$12: C18.1, U$3.CDT
- new net N$16: R53.1, U$3.VDD
- new net N$17: R54.1, U$4.VDD
- new net N$2: R47.2, U$3.CTLD
- new net N$270: D1.A, R1.1
- new net N$271: D2.A, R2.1
- new net N$3: R47.1, U$4.DO
- new net N$385: C13.1, C14.1, R39.1, U1.VBATT
- new net N$398: C4.1, Q3.S, R29.2, R35.2, U4.RS-, U7.IN
- new net N$4: R48.2, U$3.CTLC
- new net N$401: R41.2, R42.2, U1.THRM
- new net N$403: R41.1, R43.2, U1.AIN2
- new net N$404: R42.1, R44.2, U1.AIN1
- new net N$405: U1.ALRT1
- new net N$407: B3.NEG, B4.NEG, C15.2, C19.2, R40.1, R51.1, R52.1, U$4.VSS, U1.CSP
- new net N$480: TP2.1, U3.IO3
- new net N$482: TP3.1, U3.IO4
- new net N$499: C13.2, C15.1, R55.2, U1.CELL1, U1.CELL2
- new net N$5: R51.2, U$4.CDT
- new net N$518: TP4.1, U3.IO5
- new net N$523: TP5.1, U3.IO6
- new net N$573: R12.2, TP10.1, U3.IO7
- new net N$575: D4.A, R12.1
- new net N$579: C6.1, Q1.1.S, R25.2
- new net N$580: C6.2, Q1.1.G, Q1.2.D, R15.2
- new net N$581: C8.2, Q1.2.G, R16.2, R18.1
- new net N$589: R26.1, U3.!RESET
- new net N$590: Q4.G, Q5.D, R27.1
- new net N$593: Q4.D, R29.1, U4.RS+
- new net N$596: R31.1, R32.2, TP12.1, U4.CIN1+
- new net N$597: R33.1, R34.2, TP11.1, U4.CIN1-
- new net N$598: R31.2, U4.IOUT
- new net N$599: R33.2, U4.CIN2-, U4.REF
- new net N$6: R48.1, U$4.CO
- new net N$600: TP6.1, U4.POUT
- new net N$603: C2.1, R36.2, R37.2
- new net N$604: R37.1, U4.INHIBIT
- new net N$8: Q2.1.G, R50.1, U$3.DO
- new net N$9: Q2.2.G, R49.1, U$3.CO
- new net ON/!OFF: Q5.G, R28.2, TP13.1, U3.IO0
- new net PEN-SCL-FILT: R13.1, R21.1, R24.2, R6.1, TP18.1, U3.SCL
- new net PEN-SDA-FILT: Q1.1.D, R16.1, R19.2, R23.2, R9.2, TP20.1, U3.SDA
- new net SCL: R3.1, U1.OD/SCL, U6.PB6
- new net SDA: R46.1, U1.DQ/SDA, U6.PB7
- new net TPS62111-PG: TP16.1, U5.PG
- new net TPS62111-SYNC: R10.2, R7.1, TP19.1, U5.SYNC
- new net TPS62111_SW: L2.1, U5.SW
- new net VBUSP: C10.1, C2.2, C7.1, Q3.D, R1.2, R7.2, TP9.1, U5.EN, U5.VIN
- new net VPD: C1.2, C8.1, Q1.2.S, R11.2, R18.2, R20.2, R26.2, R38.2, R4.2, R5.2, TP1.1, U3.V+
- net CAN1_H: now also U2.CANH
- net CAN1_L: now also U2.CANL
- net GND: now also C1.1, C10.2, C11.2, C12.2, C14.2, C16.2, C17.1, C22.1, C3.1, C4.2, C5.2, C7.2, C9.1, D1.C, D2.C, D4.C, Q5.S, Q6.S, R10.1, R14.1, R15.1, R17.1, R22.1, R28.1, R30.1, R32.1, R34.1, R36.1, R40.2, R43.1, R44.1, R8.1, U1.CELLX, U1.CSN, U1.GND, U2.GND, U3.GND, U4.GND, U5.GND, U5.LBI, U5.LBO, U6.VSS, U7.GND, X1.SHIELD; no longer R1.1, R5.1
- net N$10: now also Q2.1.S, R39.2, R50.2; no longer Q1.D, R9.2
- net N$11: now also Q2.1.D, Q2.2.D; no longer Q2.D, R10.2
- net N$14: now also R52.2, U$4.CTLD; no longer Q3.G, R11.2, R13.1
- net N$15: now also B1.POS, B2.POS, C21.1, Q2.2.S, R49.2, R53.2; no longer Q4.G, R12.2, R14.1
- net OPD_PWR: now also R4.1
- net OPD_SCL: now also R24.1
- net OPD_SDA: now also R25.1
- net V1S: now also C18.2, C19.1, C21.2, R54.2, R55.1, U$3.VSS; no longer Q1.S, R10.1, R8.2
- net VBUS: now also Q4.S, R27.2; no longer F1.P$2
Other:
- note added: "(3.3V)"
- note added: "0402"
- note added: "0805"
- note added: "3.1"
- note added: "3.3V Card Switching Supply"
- note added: "Address selection for Card (See MAX7310 datasheet)"
- note added: "All caps are 0402 ceramic 10% X5R Vw>=16V unless marked"
- note added: "All resistors 0402 +/- 1% unless marked"
- note added: "Auxiliary Connector"
- note added: "Battery Pack"
- note added: "CAN Transceiver"
- note added: "Card Power Switch and Circuit Breaker"
- note added: "Cell Balancing/Fuel Gauge"
- note added: "ECS-MPI4040R4-6R8-R"
- note added: "Main Power Switch"
- note added: "NTC Thermistors"
- note added: "Note: Address 0b0111110x is reserved on all oresat cards"
- note added: "Note: the S8209 has capability for cell balancing that we are not utilizing in favor of the MAX17205 cell balancing"
- note added: "OreSat Power Domain (OPD) Controller"
- note added: "OreSat Power Domain (OPD) Power Supply (3.3V)"
- note added: "OreSat Power Enable (PEN)"
- note added: "OreSat Proto-Card"
- note added: "Overcharge/Discharge protection"
- note added: "Vbus = (6.0,7.2,8.4)V"
- note removed: "(49.5 88.769)"
- note removed: "1206"
- note removed: "2012"
- note removed: "2012 1/2W"
- note removed: "2A cont, 4A trip."
- note removed: "REPLACE WITH 0 OHM FOR FLIGHT"
- note removed: "thermistor"
- moved on the sheet: C1, C10, C2, C4, C5, C6, C7, C8, J6, R1, R10, R11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

Commit message: Design review of schematic. Added labels, nets to M0, shutdown circuitry, discussed power domains.
Parts:
- removed J1: J-SAMTEC-TFM-110-X1-XXX-D-RA, J-Samtec-TFM-110-X1-XXX-D-RA:J-SAMTEC-TFM-110-X1-XXX-D-RA
- removed R49: 4.7k, rcl:R-US_R0402
- removed R51, R52: 1k, rcl:R-US_R0402
- added C20: 10n, rcl_custom:C-EU0402-B-NOSILK
- added D3, D5, D6: D-0402, D-0402-package:D-0402
- added R45: 100k, rcl_custom:R-US_0402-B-NOSILK
- added TP21, TP22, TP23, TP24, TP7: TEST-POINT, Tova:TEST-POINT
- C13, C15: device oresat-rcl:C-USC0402 -> rcl_custom:C-EU0402-B-NOSILK
- C14: device oresat-rcl:C-USC0402 -> rcl_custom:C-EU0603-B-NOSILK
- C18, C19, C21: device rcl:C-USC0402K -> rcl_custom:C-EU0402-B-NOSILK
- R39: device oresat-rcl:R-US_0603-B -> rcl_custom:R-US_0402-B-NOSILK
- R41, R42: device rcl:R-US_R0603 -> rcl_custom:R-US_0402-B-NOSILK
- R47, R48, R53, R54: device rcl:R-US_R0402 -> rcl_custom:R-US_0402-B-NOSILK
- R50: value 4.7k -> 100k; device rcl:R-US_R0402 -> rcl_custom:R-US_0402-B-NOSILK
Connections:
- removed net AUX_!SHUTDOWN: J1.19, J1.20
- removed net AUX_CAN1_H: J1.13, J1.14
- removed net AUX_CAN1_L: J1.15, J1.16
- removed net AUX_CAN2_H: J1.1, J1.2
- removed net AUX_CAN2_L: J1.3, J1.4
- removed net AUX_GND1: J1.17, J1.18
- removed net AUX_GND2: J1.11, J1.12
- removed net AUX_GND3: J1.10, J1.9
- removed net AUX_VBUS1: J1.7, J1.8
- removed net AUX_VBUS2: J1.5, J1.6
- removed net N$1: R3.2, R46.2
- removed net N$10: Q2.1.S, R39.2, R50.2
- removed net N$500: J6.11, J6.12
- removed net N$503: J6.10, J6.9
- removed net N$504: J6.5, J6.6
- removed net N$519: J6.3, J6.4
- removed net N$520: J6.1, J6.2
- removed net N$524: J6.23, J6.24
- removed net N$525: J6.21, J6.22
- removed net N$528: J6.13, J6.14
- removed net SPARE4: J6.7, J6.8
- new net !CHRG-DISABLE: D6.C
- new net !SHDWN-M0: D3.C
- new net N$7: C20.1, U$4.CDT
- net !SHUTDOWN: now also D5.C
- net 3.3V: now also R3.2, R46.2
- net N$14: now also D6.A, TP22.1, U$4.CTLC; no longer R52.2, U$4.CTLD
- net N$15: now also R45.2; no longer R49.2
- net N$2: now also TP24.1
- net N$4: now also TP23.1
- net N$407: now also C20.2; no longer R51.1, R52.1
- net N$5: now also D3.A, D5.A, TP21.1, TP7.1, U$4.CTLD; no longer R51.2, U$4.CDT
- net N$9: now also R45.1; no longer R49.1
- net VBUS: now also Q2.1.S, R39.2, R50.2
Other:
- note added: "100 ms of delay"
- note added: "DOES THE CB GO TO VBUS OR TO VBAT?"
- note added: "FUSE HERE 5A 1206 or greater, like 2012?"
- note added: "WHAT ABOUT POWER DOMAINS"
- note removed: "0402"
- note removed: "Auxiliary Connector"
- moved on the sheet: B1, B2, B3, B4, C11, C16, C17, C22, C3, C9, R17, R3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
