File: eagle/oresat-batteries.sch (EAGLE design)
At the start: 300 parts, among them J2 ORESAT-DEBUG-CONNECTOR-CARD, J6 J-SAMTEC-TFM-120-X1-XXX-D-RA, Q1 BSS84, Q10 BSS84, Q11 BSS84, Q12 Si7625DN, Q13 Si7625DN, Q14 Si7625DN, Q15 Si7625DN, Q16 Si7625DN, Q17 MOSFET-PCH-SOT23-6, Q18 MOSFET-PCH-SOT23-6, Q19 PMV45EN, Q2 Si7625DN, Q20 PMV45EN, Q21 DMP2240UDM, Q23 Si7625DN, Q24 Si7625DN, Q25 BSS84, Q26 BSS84, Q27 Si7625DN, Q28 Si7625DN, Q29 Si7625DN, Q3 BSS84, Q30 Si7625DN, Q31 Si7625DN, Q32 BSS84, Q33 BSS84, Q9 Si7625DN, U10 LTC4412, U11 S-8209AAA-T8T1U, U12 S-8209AAA-T8T1U, U13 S-8209AAA-T8T1U, U14 S-8209AAA-T8T1U, U15 MAX17205G, U18 MAX7310ATE, U19 MAX4211FETE, U2 MAX17205G, U20 TPS62111RSA, U21 MIC842LYC5, U22 MIC842LYC5, U3 TCAN330, U4 STM32F042K6, U7 LTC4412, U8 LTC4412, U9 LTC4412, X2 16MHZ-2.5x2mm

Commit message: Now with 100% realistic SOT23-3 transistors and more cleanup.
Parts:
- removed D1, D12, D4, D9: (no value), diode:DIODE-SOD123
- removed F3: (no value), oresat-rcl:R-US_1206-C
- removed R8, R87: 10k, oresat-rcl:R-US_0603-C-NOSILK
- removed T20, T4: (no value), zetex:NMOSSOT23
- added F2: GENERIC-FUSE-1206, F-Generic-Fuse-1206:GENERIC-FUSE-1206
- F1: value (none) -> GENERIC-FUSE-1206; device oresat-rcl:R-US_1206-C -> F-Generic-Fuse-1206:GENERIC-FUSE-1206
- Q1, Q10, Q11, Q25, Q26, Q3, Q32, Q33: value BSS84 -> NTR4101; device Transistor:BSS84 -> Q-MOSFET-PCH-SOT23-3:P-MOSFET-SOT23-3
- Q19, Q20: device Tova:PMV45EN -> Q-MOSFET-NCH-SOT23-3:N-MOSFET-SOT-23-3
- R126: device rcl:R-US_R1206 -> oresat-rcl:R-US_1206-C
- T1, T17, T18, T19, T21, T22, T23, T24, T3, T5, T6: value (none) -> PM45VEN; device zetex:NMOSSOT23 -> Q-MOSFET-NCH-SOT23-3:N-MOSFET-SOT-23-3
- T2, T7, T8: value (none) -> PMV45EN; device zetex:NMOSSOT23 -> Q-MOSFET-NCH-SOT23-3:N-MOSFET-SOT-23-3
Connections:
- removed net N$1: D1.C, D4.C, T4.D
- removed net N$92: D12.C, D9.C, T20.D
- removed net OPD-PK1-DISABLE: R8.2, T4.G
- removed net OPD-PK2-DISABLE: R87.2, T20.G
- net CSP-PK1: no longer R8.1, T4.S
- net CSP-PK2: no longer R87.1, T20.S
- net N$11: no longer D4.A
- net N$51: no longer D1.A
- net N$77: no longer D12.A
- net N$91: no longer D9.A
- net VBATT-F-PK1: now also F1.P$1; no longer F1.2
- net VBATT-F-PK2: now also F2.P$1; no longer F3.2
- net VBATT-PK1: now also F1.P$2; no longer F1.1
- net VBATT-PK2: now also F2.P$2; no longer F3.1
Other:
- note added: "ALL CAPS ARE 0603, 10%, X5R, WV >= 16 V UNLESS OTHERWISE NOTED ALL RESISTORS ARE 0603 1% UNLESS OTHERWISE NOTED"
- note added: "Battery Board outline:"
- note added: "Microcontroller and OPD based on v3.4."
- note added: "OreSat battery Card - Connectors"
- note removed: "ALL CAPS ARE 0603 5% WITH WV >= 16 V UNLESS OTHERWISE NOTED ALL RESISTORS ARE 0603 1% UNLESS OTHERWISE NOTED"
- note removed: "All caps are 0402 ceramic 10% X5R Vw>=16V unless marked"
- note removed: "All resistors 0402 +/- 1% unless marked"
- note removed: "Based on Protocard v3.4"
- note removed: "FIXME"
- note removed: "Include Battery Board outline"
- note removed: "OreSat battery Card - Microcontroller"
- note removed: "The battery pack is disconnected if OPD-PK1_DISABLE is asserted - will neither charge nor discharge."
- moved on the sheet: B1, B2, B3, B4, C17, C22, C23, C24, C25, C26, C27, C28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

Commit message: Renumbered parts using built-in renumber tool.
Parts:
- removed C37: 100n, oresat-rcl:C-EU0603-C-NOSILK
- removed C38: NP, oresat-rcl:C-EU0603-C-NOSILK
- removed C40: 1u, oresat-rcl:C-EU0603-C-NOSILK
- removed C41: 22u, oresat-rcl:C-EU0805-B-NOSILK
- removed D14: GREEN, SparkFun-LED:LED-GREEN0603
- removed R107: 2.7k, oresat-rcl:R-US_0603-C-NOSILK
- removed R109: 10, oresat-rcl:R-US_0603-C-NOSILK
- removed R110, R111, R113, R114, R117, R118, R119, R121: NP, oresat-rcl:R-US_0603-C-NOSILK
- removed R122, R142: 100, oresat-rcl:R-US_0603-C-NOSILK
- removed R123, R139: 10k, oresat-rcl:R-US_0603-C-NOSILK
- removed T17, T19, T21, T22, T23, T5: PM45VEN, Q-MOSFET-NCH-SOT23-3:N-MOSFET-SOT-23-3
- removed T2, T7: PMV45EN, Q-MOSFET-NCH-SOT23-3:N-MOSFET-SOT-23-3
- removed TP72, TP73, TP75, TP76, TP79, TP80, TP82, TP83, TP84, TP85, TP86, TP87, TP88, TP89: TEST-POINT-LARGE-SQUARE, oresat-misc:TEST-POINT-LARGE-SQUARE
- removed U19: MAX4211FETE, U-Maxim-MAX4211-power-monitor:MAX4211
- removed U21, U22: MIC842LYC5, U-Microchip-MIC842-Comparator:MIC842LYC5
- added C11: 100n, oresat-rcl:C-EU0603-C-NOSILK
- added C16: 10n, oresat-rcl:C-EU0603-C-NOSILK
- added C35, C36: 470n, oresat-rcl:C-EU0603-C-NOSILK
- added D4: GREEN, SparkFun-LED:LED-GREEN0603
- added Q34, Q35, Q36, Q37, Q38: Si7625DN, Q-VIshay-MOSFET-PCH-PowerPak121-8:Q-VISHAY-MOSFET-PCH-POWERPAK-1212-8
- added Q4: DMP3050LVT-7, Q-MOSFET-PCH-SOT23-6:MOSFET-PCH-SOT23-6
- added Q41: NTR4101, Q-MOSFET-PCH-SOT23-3:P-MOSFET-SOT23-3
- added Q5: PMV45EN, Q-MOSFET-NCH-SOT23-3:N-MOSFET-SOT-23-3
- added R100, R101, R102, R103, R104, R99: 10k, oresat-rcl:R-US_0603-C-NOSILK
- added R46, R49: 1M, oresat-rcl:R-US_0603-C-NOSILK
- added R87, R94, R97, R98: 100k, oresat-rcl:R-US_0603-C-NOSILK
- added R95: 10, oresat-rcl:R-US_0603-C-NOSILK
- added R96: 100, oresat-rcl:R-US_0603-C-NOSILK
- added TP19, TP20, TP26, TP38, TP39, TP40, TP41, TP42, TP43, TP44, TP45, TP46, TP70, TP71: TEST-POINT-LARGE-SQUARE, oresat-misc:TEST-POINT-LARGE-SQUARE
- added U16: LTC4412, U-LT-LTC4412-ideal-diode:LTC4412
- added U17: MAX17205G, U-Maxim-MAX17205-Fuel_Gauge:MAX17205G
- added U6: TCAN330, TCAN330:TCAN330
- C10: value 20p -> 100n; DPN 1276-6601-1-ND -> 1276-1001-1-ND; MPN CL05C200JB51PNC -> CL05B104KO5NNNC
- C13: value 1n -> 20p; DIS (none) -> Digi-Key; DPN (none) -> 1276-6601-1-ND; MFR (none) -> Samsung; MPN (none) -> CL05C200JB51PNC
- C14: value 100n -> 20p; DIS (none) -> Digi-Key; DPN (none) -> 1276-6601-1-ND; MFR (none) -> Samsung; MPN (none) -> CL05C200JB51PNC
- C15, C17, C23: value 1n -> 100n
- C20: value 10n -> 1n
- C21, C31: value 100n -> 1n
- C24: value 10n -> 470n
- C25: value 100n -> 470n
- C29: value 100n -> 10n
- C3, C9: value 470n -> 100n; DIS (none) -> Digi-Key; DPN (none) -> 1276-1001-1-ND; MFR (none) -> Samsung; MPN (none) -> CL05B104KO5NNNC
- C32: value 470n -> 1n
- C33: value 470n -> 100n
- C34: DIS Digi-Key -> (none); DPN 1276-1001-1-ND -> (none); MFR Samsung -> (none); MPN CL05B104KO5NNNC -> (none)
- C6: value 100n -> 1u; DPN 1276-1001-1-ND -> 311-1446-1-ND; MFR Samsung -> Yageo; MPN CL05B104KO5NNNC -> CC0603KRX7R7BB105
- C7: value 100n -> NP; DIS Digi-Key -> (none); DPN 1276-1001-1-ND -> (none); MFR Samsung -> (none); MPN CL05B104KO5NNNC -> (none)
- C8: value 20p -> 22u; device oresat-rcl:C-EU0603-C-NOSILK -> oresat-rcl:C-EU0805-B-NOSILK; DPN 1276-6601-1-ND -> 490-9959-1-ND; MFR Samsung -> Murata; MPN CL05C200JB51PNC -> GRM21BD71A226ME44L
- D1: value AMBER -> GREEN
- D2: value AMBER -> GREEN; DPN 1830-1064-1-ND -> 511-1584-1-ND; MFR Inolux -> Rohm; MPN IN-S63AT5A -> SML-E12M8WT86
- Q1: value NTR4101 -> DMP2240UDM; device Q-MOSFET-PCH-SOT23-3:P-MOSFET-SOT23-3 -> Q-MOSFET-PCH-dual-SOT23-6:MOSFET-PCH-SOT23-6; DIS (none) -> Digi-Key; DPN (none) -> DMP2240UDMDICT-ND; MFR (none) -> Diodes Inc; MPN (none) -> DMP2240UDM
- Q11: value NTR4101 -> PMV45EN; device Q-MOSFET-PCH-SOT23-3:P-MOSFET-SOT23-3 -> Q-MOSFET-NCH-SOT23-3:N-MOSFET-SOT-23-3
- Q14, Q15, Q23, Q28: value Si7625DN -> NTR4101; device Q-VIshay-MOSFET-PCH-PowerPak121-8:Q-VISHAY-MOSFET-PCH-POWERPAK-1212-8 -> Q-MOSFET-PCH-SOT23-3:P-MOSFET-SOT23-3
- Q17, Q18: value MOSFET-PCH-SOT23-6 -> Si7625DN; device Q-MOSFET-PCH-SOT23-6:MOSFET-PCH-SOT23-6 -> Q-VIshay-MOSFET-PCH-PowerPak121-8:Q-VISHAY-MOSFET-PCH-POWERPAK-1212-8; DIS Digi-Key -> (none); DPN DMP3050LVT-7DICT-ND -> (none); MFR Diodes Inc -> (none); MPN DMP3050LVT-7 -> (none)
- Q19, Q20: value PMV45EN -> Si7625DN; device Q-MOSFET-NCH-SOT23-3:N-MOSFET-SOT-23-3 -> Q-VIshay-MOSFET-PCH-PowerPak121-8:Q-VISHAY-MOSFET-PCH-POWERPAK-1212-8; DIS Digi-Key -> (none); DPN 1727-2307-1-ND -> (none); MFR Nexperia -> (none); MPN PMV45EN2R -> (none)
- Q2: value Si7625DN -> PMV45EN; device Q-VIshay-MOSFET-PCH-PowerPak121-8:Q-VISHAY-MOSFET-PCH-POWERPAK-1212-8 -> Q-MOSFET-NCH-SOT23-3:N-MOSFET-SOT-23-3; DIS (none) -> Digi-Key; DPN (none) -> 1727-2307-1-ND; MFR (none) -> Nexperia; MPN (none) -> PMV45EN2R
- Q21: value DMP2240UDM -> PMV45EN; device Q-MOSFET-PCH-dual-SOT23-6:MOSFET-PCH-SOT23-6 -> Q-MOSFET-NCH-SOT23-3:N-MOSFET-SOT-23-3; DIS Digi-Key -> (none); DPN DMP2240UDMDICT-ND -> (none); MFR Diodes Inc -> (none); MPN DMP2240UDM -> (none)
- Q24, Q27, Q29, Q9: value Si7625DN -> PM45VEN; device Q-VIshay-MOSFET-PCH-PowerPak121-8:Q-VISHAY-MOSFET-PCH-POWERPAK-1212-8 -> Q-MOSFET-NCH-SOT23-3:N-MOSFET-SOT-23-3
- Q25, Q26: value NTR4101 -> PM45VEN; device Q-MOSFET-PCH-SOT23-3:P-MOSFET-SOT23-3 -> Q-MOSFET-NCH-SOT23-3:N-MOSFET-SOT-23-3
- Q3: value NTR4101 -> DMP3050LVT-7; device Q-MOSFET-PCH-SOT23-3:P-MOSFET-SOT23-3 -> Q-MOSFET-PCH-SOT23-6:MOSFET-PCH-SOT23-6; DIS (none) -> Digi-Key; DPN (none) -> DMP3050LVT-7DICT-ND; MFR (none) -> Diodes Inc; MPN (none) -> DMP3050LVT-7
- R1: value 10k -> 10; DIS (none) -> Digi-Key; DPN (none) -> 311-100LRCT-ND; MFR (none) -> Yageo; MPN (none) -> RC0402FR-07100RL
- R10, R2, R3, R4, R9: value 10k -> NP; DIS (none) -> Digi-Key; DPN (none) -> 1276-4275-1-ND; MFR (none) -> Samsung; MPN (none) -> RC1005F6653CS
- R14: value 2.7k -> NP; DPN A129632CT-ND -> 1276-4275-1-ND; MFR TE Connectivity -> Samsung; MPN CRGCQ0402F2K7 -> RC1005F6653CS
- R15: value 10k -> NP; DPN 311-10.0KLRCT-ND -> 1276-4275-1-ND; MFR Yageo -> Samsung; MPN RC0402FR-0710KL -> RC1005F6653CS
- R16: value 4.7k -> NP; DPN A129632CT-ND -> 1276-4275-1-ND; MFR TE Connectivity -> Samsung; MPN CRGCQ0402F2K7 -> RC1005F6653CS
- R18: value 4.7k -> 10k; DPN A129632CT-ND -> 311-10.0KLRCT-ND; MFR TE Connectivity -> Yageo; MPN CRGCQ0402F2K7 -> RC0402FR-0710KL
- R39: value 10 -> 2.7k; DIS (none) -> Digi-Key; DPN (none) -> A129632CT-ND; MFR (none) -> TE Connectivity; MPN (none) -> CRGCQ0402F2K7
- R40: value 10m -> 10k; device oresat-rcl:R-US_1206-C -> oresat-rcl:R-US_0603-C-NOSILK; DIS (none) -> Digi-Key; DPN (none) -> 311-10.0KLRCT-ND; MFR (none) -> Yageo; MPN (none) -> RC0402FR-0710KL
- R41: value 10k -> 2.7k; DIS (none) -> Digi-Key; DISTRIBUTOR Digi-key -> (none); DPN RNCP0603FTD10K0CT-ND -> A129632CT-ND; MFR (none) -> TE Connectivity; MPN RNCP0603FTD10K0 -> CRGCQ0402F2K7
- R42: DIS (none) -> Digi-Key; DPN (none) -> 311-10.0KLRCT-ND; MFR (none) -> Yageo; MPN (none) -> RC0402FR-0710KL
- R43, R44: value 10k -> 4.7k; DIS (none) -> Digi-Key; DPN (none) -> A129632CT-ND; MFR (none) -> TE Connectivity; MPN (none) -> CRGCQ0402F2K7
- R45, R83: value 100k -> 1k
- R47, R85: value 1k -> 10k
- R50, R73, R74, R77: value 100k -> 10k
- R51: value 10 -> 470
- R52: value 10m -> 1k; device oresat-rcl:R-US_1206-C -> oresat-rcl:R-US_0603-C-NOSILK
- R53: value 470 -> 1k
- R55: value 100 -> 10k
- R56: DISTRIBUTOR Digi-key -> (none); DPN RNCP0603FTD10K0CT-ND -> (none); MPN RNCP0603FTD10K0 -> (none)
- R57: value 10k -> 100k
- R58, R59, R88, R89, R90, R91: value 10k -> 1M
- R6: value 1k -> 100; DIS (none) -> Digi-Key; DPN (none) -> 311-100LRCT-ND; MFR (none) -> Yageo; MPN (none) -> RC0402FR-07100RL
- R60, R61: value 470 -> 1M
- R62: value 1k -> 10m; device oresat-rcl:R-US_0603-C-NOSILK -> oresat-rcl:R-US_1206-C
- R63: value 1k -> 100; device oresat-rcl:R-US_0603-C-NOSILK -> oresat-rcl:R-US_1206-C
- R64: value 100 -> 100k
- R65: value 100k -> 10
- R66: value 1k -> 100
- R67, R68: value 1M -> 100k
- R69, R72, R80, R86: value 1M -> 10k
- R7: value 1M -> 100; DIS (none) -> Digi-Key; DPN (none) -> 311-100LRCT-ND; MFR (none) -> Yageo; MPN (none) -> RC0402FR-07100RL
- R70: value 100 -> 10k; device oresat-rcl:R-US_1206-C -> oresat-rcl:R-US_0603-C-NOSILK
- R71: value 1M -> 10k; DISTRIBUTOR (none) -> Digi-key; DPN (none) -> RNCP0603FTD10K0CT-ND; MPN (none) -> RNCP0603FTD10K0
- R78: value 1M -> 1k
- R81: value 1M -> 470
- R82: value 100 -> 1k; device oresat-rcl:R-US_1206-C -> oresat-rcl:R-US_0603-C-NOSILK
- R84: value 100k -> 470
- R92: value 10k -> 10m; device oresat-rcl:R-US_0603-C-NOSILK -> oresat-rcl:R-US_1206-C
- R93: value 10k -> 100; device oresat-rcl:R-US_0603-C-NOSILK -> oresat-rcl:R-US_1206-C
- U11: value S-8209AAA-T8T1U -> LTC4412; device U-ABLIC-s8209A-BattProtection:S-8209AXXT -> U-LT-LTC4412-ideal-diode:LTC4412; MFR Ablic -> (none); MPN S-8209AAA-T8T1U -> (none)
- U12: value S-8209AAA-T8T1U -> MAX17205G; device U-ABLIC-s8209A-BattProtection:S-8209AXXT -> U-Maxim-MAX17205-Fuel_Gauge:MAX17205G; MFR Ablic -> (none); MPN S-8209AAA-T8T1U -> (none)
- U15: value MAX17205G -> LTC4412; device U-Maxim-MAX17205-Fuel_Gauge:MAX17205G -> U-LT-LTC4412-ideal-diode:LTC4412
- U2: value MAX17205G -> MIC842LYC5; device U-Maxim-MAX17205-Fuel_Gauge:MAX17205G -> U-Microchip-MIC842-Comparator:MIC842LYC5
- U3: value TCAN330 -> MIC842LYC5; device TCAN330:TCAN330 -> U-Microchip-MIC842-Comparator:MIC842LYC5; DIS Digi-Key -> (none); DPN 296-44211-1-ND -> (none); MFR Texas Instruments -> (none); MPN TCAN330GDCNT -> (none)
- U4: value STM32F042K6 -> MAX4211FETE; device STM32F042K:STM32F042K6 -> U-Maxim-MAX4211-power-monitor:MAX4211; DPN 497-18516-ND -> MAX4211FETE+-ND; MFR STMicroelectronics -> Maxim; MPN STM32F042K6T7 -> MAX4211FETE
- U7: value LTC4412 -> STM32F042K6; device U-LT-LTC4412-ideal-diode:LTC4412 -> STM32F042K:STM32F042K6; DIS (none) -> Digi-Key; DPN (none) -> 497-18516-ND; MFR (none) -> STMicroelectronics; MPN (none) -> STM32F042K6T7
- U8, U9: value LTC4412 -> S-8209AAA-T8T1U; device U-LT-LTC4412-ideal-diode:LTC4412 -> U-ABLIC-s8209A-BattProtection:S-8209AXXT; MFR (none) -> Ablic; MPN (none) -> S-8209AAA-T8T1U
- renumbered C39 to C5, C42 to C4, C43 to C2, C44 to C1, D10 to D6, D11 to D5, D13 to D3, D15 to D1, J6 to J1, JP5 to JP4, JP6 to JP3, R108 to R36, R112 to R17, R115 to R8, R116 to R11, R120 to R5, R124 to R25, R125 to R24, R126 to R30, R127 to R31, R128 to R33, R129 to R35, R130 to R32, R131 to R34, R132 to R37, R133 to R26, R134 to R27, R135 to R38, R136 to R28, R137 to R29, R138 to R23, R140 to R20, R141 to R22, R143 to R12, R144 to R19, R145 to R21, T1 to Q8, T18 to Q39, T24 to Q40, T3 to Q6, T6 to Q7, T8 to Q22, TP74 to TP16, TP77 to TP17, TP78 to TP18, TP81 to TP15, U18 to U1, U20 to U5, X2 to X1
Connections:
- removed net N$76 (its old number): Q27.S, Q28.S
- new net N$81: Q36.S, Q37.S
- net !CHARGE-PK1: now also Q23.G, R69.1, TP33.1, U9.CO; no longer Q3.G, R3.1, TP9.1, U11.CO
- net !CHARGE-PK2: now also Q41.G, R99.1, TP56.1, U14.CO; no longer Q33.G, R92.1, TP64.1, U13.CO
- net !DISCHARGE-PK1: now also Q10.G, R56.1, TP32.1, U9.DO; no longer Q1.G, R1.1, TP10.1, U11.DO
- net !DISCHARGE-PK2: now also Q28.G, R86.1, TP55.1, U14.DO; no longer Q32.G, R90.1, TP65.1, U13.DO
- net !FAST-CHARGE-PK1: now also Q20.G, Q21.D, R64.2; no longer Q14.G, R73.2, T2.D
- net !FAST-CHARGE-PK2: now also Q38.G, R94.2; no longer Q29.G, R83.2
- net !FAULT: now also Q5.D; no longer Q20.D
- net !SD: now also TP34.1, TP57.1; no longer TP11.1, TP66.1
- net 3.3V: now also C10.2, C11.2, C8.1, C9.2, R43.2, R44.2, U6.VCC, U7.VDD, U7.VDDA, U7.VDDIO2; no longer C34.2, C41.1, C6.2, C7.2, R16.2, R18.2, U3.VCC, U4.VDD, U4.VDDA, U4.VDDIO2
- net AD0: now also R14.2, R15.1, R16.1; no longer R110.1, R111.2, R113.1
- net AD1: now also R10.1, R9.1; no longer R114.1, R117.1
- net AD2: now also R2.2, R3.1, R4.1; no longer R118.1, R119.2, R121.1
- net AIN1-PK1: now also JP2.1, R73.1, R74.2, U12.AIN1; no longer JP1.1, R42.1, R44.2, U2.AIN1
- net AIN1-PK2: now also R103.1, R104.2, U17.AIN1; no longer R57.1, R59.2, U15.AIN1
- net AIN2-PK1: now also JP1.1, R71.1, R72.2, U12.AIN2; no longer JP2.1, R41.1, R43.2, U2.AIN2
- net AIN2-PK2: now also R101.1, R102.2, U17.AIN2; no longer R56.1, R58.2, U15.AIN2
- net ALERTA-PK1: now also TP48.1, U12.ALRT1, U7.PB5; no longer TP28.1, U2.ALRT1, U4.PB5
- net ALERTA-PK2: now also TP71.1, U17.ALRT1, U7.PB1; no longer TP52.1, U15.ALRT1, U4.PB1
- net BOOT0: now also R41.2, R42.2, TP24.1, U7.PB8-BOOT0; no longer R13.2, R14.2, TP27.1, U4.PB8-BOOT0
- net CAN1_H: now also U6.CANH; no longer U3.CANH
- net CAN1_L: now also U6.CANL; no longer U3.CANL
- net CAN_RX: now also U6.RXD, U7.PA11; no longer U3.RXD, U4.PA11
- net CAN_SHDN: now also U6.SHDN, U7.PA10; no longer U3.SHDN, U4.PA10
- net CAN_SILENT: now also U6.S, U7.PA9; no longer U3.S, U4.PA9
- net CAN_TX: now also U6.TXD, U7.PA12; no longer U3.TXD, U4.PA12
- net CB-RESET: now also TP14.1, U4.CIN2-; no longer TP76.1, U19.CIN2-
- net CB_CTRL: now also Q4.G, Q5.G, TP9.1, U4.COUT1, U4.COUT2, U4.LE; no longer Q17.G, Q20.G, TP86.1, U19.COUT1, U19.COUT2, U19.LE
- net CELL1-PK1: now also C20.2, C21.1, R66.2, TP46.1, U12.CELL1, U12.CELL2; no longer C13.2, C15.1, R55.2, TP25.1, U2.CELL1, U2.CELL2
- net CELL1-PK2: now also C31.2, C32.1, R96.2, TP69.1, U17.CELL1, U17.CELL2; no longer C17.2, C23.1, R64.2, TP51.1, U15.CELL1, U15.CELL2
- net CHARGE-DISABLE-PK1: now also R47.2, U7.PA15; no longer R9.2, U4.PA15
- net CHARGE-DISABLE-PK2: now also Q25.G, R77.2, U7.PA6; no longer R88.2, T22.G, U4.PA6
- net CHARGE-STAT-OC-PK1: now also TP45.1, U11.STAT, U7.PA0; no longer TP37.1, U10.STAT, U4.PA0
- net CHARGE-STAT-OC-PK2: now also TP68.1, U16.STAT, U7.PA4; no longer TP55.1, U4.PA4, U8.STAT
- net CRYSTALIN1: now also C14.1, U7.PF0-OSC_IN; no longer C10.1, U4.PF0-OSC_IN
- net CRYSTALOUT1: now also C13.1, U7.PF1-OSC_OUT; no longer C8.1, U4.PF1-OSC_OUT
- net CSP-PK1: now also C16.2, C21.2, Q9.S, R47.1, R50.1, R61.2, R62.1, TP42.1, U12.CSP, U8.VSS; no longer C19.2, C20.2, R10.1, R40.1, R68.2, R9.1, T5.S, TP3.1, U12.VSS, U2.CSP
- net CSP-PK2: now also B4.NEG, C32.2, Q24.S, Q25.S, Q26.S, Q27.S, R77.1, R80.1, R91.2, R92.1, TP65.1, U13.VSS, U17.CSP; no longer B3.NEG, C23.2, R52.1, R78.2, R88.1, R89.1, T17.S, T19.S, T21.S, T22.S, TP58.1, U14.VSS, U15.CSP
- net DCHG-STAT-OC-PK1: now also TP35.1, U10.STAT, U7.PA1; no longer TP36.1, U4.PA1, U9.STAT
- net DCHG-STAT-OC-PK2: now also TP58.1, U15.STAT, U7.PA5; no longer TP54.1, U4.PA5, U7.STAT
- net DISCHARGE-DISABLE-PK1: now also Q9.G, R50.2, U7.PB3; no longer R10.2, T5.G, U4.PB3
- net DISCHARGE-DISABLE-PK2: now also Q27.G, R80.2, U7.PA7; no longer R89.2, T21.G, U4.PA7
- net FAST-CHARGE-PK1: now also Q21.G, R68.1, TP47.1, U7.PB4; no longer R74.1, T2.G, TP12.1, U4.PB4
- net FAST-CHARGE-PK2: now also R98.1, TP70.1, U7.PB0; no longer R84.1, TP67.1, U4.PB0
- net GND: now also C10.1, C11.1, C13.2, C19.2, C23.2, C24.2, C25.2, C3.1, C34.2, C35.2, C36.2, C6.2, C9.1, D4.C, Q11.S, Q2.S, Q21.S, Q29.S, Q5.S, R100.1, R102.1, R104.1, R42.1, R55.1, R62.2, R68.2, R70.1, R72.1, R74.1, R85.1, R92.2, R98.2, TP43.1, TP66.1, U11.GND, U12.CSN, U15.GND, U16.GND, U17.CSN, U2.GND, U4.GND, U6.GND, U7.VSS; no longer C10.2, C28.2, C29.2, C3.2, C31.2, C32.2, C34.1, C37.1, C40.2, C41.2, C6.1, C7.1, C9.2, D14.C, Q19.S, Q20.S, R139.1, R2.1, R4.1, R40.2, R43.1, R44.1, R52.2, R58.1, R59.1, R74.2, R84.2, R91.1, R93.1, T2.S, T23.S, T7.S, TP1.1, TP57.1, U15.CSN, U19.GND, U2.CSN, U21.GND, U22.GND, U4.VSS, U7.GND, U8.GND, U9.GND
- net IOUT1: now also U4.IOUT; no longer U19.IOUT
- net N$10: now also R45.1; no longer R6.1
- net N$11: now also Q9.D, R49.2, TP29.1; no longer R67.2, T5.D, TP35.1
- net N$12: now also U9.CDT; no longer U11.CDT
- net N$14: now also R45.2, TP26.1, U8.CTLC; no longer R6.2, TP22.1, U12.CTLC
- net N$15: now also Q14.D, Q16.G, R60.1; no longer Q10.D, Q9.G, R69.1
- net N$16: now also R54.1, U9.VDD; no longer R53.1, U11.VDD
- net N$17: now also R51.1, U8.VDD; no longer R54.1, U12.VDD
- net N$19: now also R39.1; no longer R107.1
- net N$2: now also R53.2, TP31.1, U9.CTLD; no longer R47.2, TP24.1, U11.CTLD
- net N$20: now also D2.A; no longer D14.A
- net N$21: now also R18.1; no longer R123.1
- net N$22: now also R67.1, U11.CTL; no longer R50.1, U10.CTL
- net N$23: now also Q2.D, Q3.G; no longer Q18.G, Q19.D
- net N$24: now also Q3.D, U4.RS+; no longer Q18.D, U19.RS+
- net N$25: now also D4.A, R41.1; no longer D2.A, R14.1
- net N$26: now also TP23.1; no longer TP33.1
- net N$27: now also TP22.1; no longer TP32.1
- net N$28: now also TP21.1; no longer TP31.1
- net N$29: now also TP20.1; no longer TP30.1
- net N$3: now also R53.1, U8.DO; no longer R47.1, U12.DO
- net N$30: now also TP19.1; no longer TP34.1
- net N$32: now also U4.CIN1+; no longer U19.CIN1+
- net N$33: now also TP13.1, U4.CIN1-; no longer TP73.1, U19.CIN1-
- net N$34: now also U4.CIN2+, U4.REF; no longer U19.CIN2+, U19.REF
- net N$35: now also U4.INHIBIT; no longer U19.INHIBIT
- net N$36: now also C7.1; no longer C38.1
- net N$37: now also R48.2, TP28.1, U8.CTLD; no longer R66.2, TP21.1, U12.CTLD
- net N$38: now also Q4.S, U4.RS-; no longer Q17.S, U19.RS-
- net N$4: now also R52.2, TP30.1, U9.CTLC; no longer R48.2, TP23.1, U11.CTLC
- net N$40: now also Q15.G, R59.2; no longer Q11.G, R71.2
- net N$41: now also Q19.D, Q20.S, Q23.S, R63.1, R64.1, R67.2, R69.2, TP44.1, U11.SENSE; no longer Q14.S, Q16.D, Q3.S, R3.2, R50.2, R70.1, R73.1, TP8.1, U10.SENSE
- net N$42: now also Q14.S, Q16.S, R58.2, TP39.1; no longer Q10.S, Q9.S, R72.2, TP14.1
- net N$43: now also Q18.G, Q19.G, U11.GATE; no longer Q15.G, Q16.G, U10.GATE
- net N$44: now also Q18.S, Q19.S; no longer Q15.S, Q16.S
- net N$45: now also Q1.1.S, R7.2; no longer Q21.1.S, R122.2
- net N$46: now also Q15.D, Q17.G, R61.1; no longer Q11.D, Q2.G, R68.1
- net N$47: now also Q1.1.G, R13.2, TP7.1, U3.OUT; no longer Q21.1.G, R139.2, TP88.1, U22.OUT
- net N$48: now also Q10.D, Q11.G, R55.2; no longer Q1.D, R2.2, T7.G
- net N$49: now also TP5.1; no longer TP87.1
- net N$5: now also R48.1; no longer R66.1
- net N$50: now also Q14.G, R58.1; no longer Q10.G, R72.1
- net N$51: now also R46.1, TP27.1; no longer R7.1, TP2.1
- net N$52: now also Q1.2.S, R6.2; no longer Q21.2.S, R142.2
- net N$53: now also Q15.S, Q17.S, R59.1, TP41.1; no longer Q11.S, Q2.S, R71.1, TP13.1
- net N$54: now also C15.1, C17.2, Q17.D, R46.2, R49.1, R51.2, R60.2, R66.1, TP40.1, U9.VSS; no longer C19.1, C21.2, Q2.D, R54.2, R55.1, R67.1, R69.2, R7.2, TP4.1, U11.VSS
- net N$56: now also Q23.D, R70.2; no longer Q3.D, R4.2
- net N$57: now also Q1.2.G, TP6.1, U2.OUT; no longer Q21.2.G, TP89.1, U21.OUT
- net N$58: now also U2.INP; no longer U21.INP
- net N$59: now also U3.INP; no longer U22.INP
- net N$6: now also R52.1, U8.CO; no longer R48.1, U12.CO
- net N$60: now also TP4.1; no longer TP83.1
- net N$65: now also R83.1, U13.DO; no longer R62.1, U14.DO
- net N$66: now also R82.1, U13.CO; no longer R63.1, U14.CO
- net N$67: now also R83.2, TP54.1, U14.CTLD; no longer R62.2, TP50.1, U13.CTLD
- net N$68: now also R82.2, TP53.1, U14.CTLC; no longer R63.2, TP49.1, U13.CTLC
- net N$69: now also R75.2, TP49.1, U13.CTLC; no longer R85.2, TP48.1, U14.CTLC
- net N$7: now also C16.1, U8.CDT; no longer C20.1, U12.CDT
- net N$70: now also R84.1, U14.VDD; no longer R60.1, U13.VDD
- net N$71: now also R81.1, U13.VDD; no longer R61.1, U14.VDD
- net N$72: now also C29.1, U14.CDT; no longer C24.1, U13.CDT
- net N$73: now also U13.CDT; no longer U14.CDT
- net N$74: now also Q30.G, Q31.G, U15.GATE; no longer Q27.G, Q28.G, U7.GATE
- net N$77: now also Q26.G, Q27.D, R79.2, TP52.1; no longer R76.2, T17.G, T21.D, TP53.1
- net N$78: now also R78.2, TP51.1, U13.CTLD; no longer R75.2, TP47.1, U14.CTLD
- net N$79: now also Q26.D, R78.1; no longer R75.1, T17.D
- net N$8: now also U10.GATE; no longer U9.GATE
- net N$80: now also Q36.G, Q37.G, U16.GATE; no longer Q30.G, Q31.G, U8.GATE
- net N$82: now also B3.POS, Q32.S, Q34.S, R88.2, TP62.1; no longer B4.POS, Q24.S, Q25.S, R81.2, TP69.1
- net N$83: now also Q33.D, Q35.G, R91.1; no longer Q23.G, Q26.D, R78.1
- net N$84: now also D8.A, Q33.G, R89.2; no longer D7.A, Q26.G, R80.2
- net N$85: now also B4.POS, Q33.S, Q35.S, R89.1, TP64.1; no longer B3.POS, Q23.S, Q26.S, R80.1, TP68.1
- net N$86: now also Q32.D, Q34.G, R90.1; no longer Q24.G, Q25.D, R79.1
- net N$87: now also D7.A, Q32.G, R88.1; no longer D8.A, Q25.G, R81.1
- net N$88: now also B3.NEG, C28.2, C29.2, Q35.D, R76.2, R79.1, R81.2, R90.2, R96.1, TP63.1, U14.VSS; no longer B4.NEG, C24.2, C25.2, Q23.D, R61.2, R64.1, R76.1, R79.2, R86.2, TP59.1, U13.VSS
- net N$89: now also Q37.D, Q38.S, Q41.S, R93.1, R94.1, R97.2, R99.2, TP67.1, U16.SENSE; no longer Q29.S, Q31.D, Q33.S, R77.2, R82.1, R83.1, R92.2, TP63.1, U8.SENSE
- net N$90: now also Q24.D, R75.1; no longer R85.1, T19.D
- net N$91: now also Q24.G, Q25.D, R76.1, TP50.1; no longer R86.1, T19.G, T22.D, TP56.1
- net N$93: now also Q28.D, Q29.G, R85.2; no longer Q32.D, R91.2, T23.G
- net N$94: now also R97.1, U16.CTL; no longer R77.1, U8.CTL
- net N$95: now also Q41.D, R100.2; no longer Q33.D, R93.2
- net NLEKJRWER: now also Q11.D, R57.1, U10.CTL; no longer R45.1, T7.D, U9.CTL
- net NLEKJRWER2: now also Q29.D, R87.1, U15.CTL; no longer R65.1, T23.D, U7.CTL
- net NRESET: now also TP25.1, U7.NRST; no longer TP29.1, U4.NRST
- net ON/!OFF: now also Q2.G, TP8.1, U4.VCC; no longer Q19.G, TP75.1, U19.VCC
- net OPD_PWR: now also R1.1; no longer R109.1
- net OPD_SCL: now also R6.1; no longer R142.1
- net OPD_SDA: now also R7.1; no longer R122.1
- net PA2/USART2_TX: now also U7.PA2; no longer U4.PA2
- net PA3/USART2_RX: now also U7.PA3; no longer U4.PA3
- net PB6/SCL: now also R44.1, U12.SCL, U17.SCL, U7.PB6; no longer R18.1, U15.SCL, U2.SCL, U4.PB6
- net PB7/SDA: now also R43.1, U12.SDA, U17.SDA, U7.PB7; no longer R16.1, U15.SDA, U2.SDA, U4.PB7
- net PEN-SCL-FILT: now also Q1.2.D, R14.1, R2.1, TP2.1; no longer Q21.2.D, R111.1, R119.1, TP84.1
- net PEN-SDA-FILT: now also Q1.1.D, R10.2, R16.2, R4.2, TP3.1; no longer Q21.1.D, R113.2, R117.2, R121.2, TP85.1
- net POUT: now also R40.1, TP11.1, U4.POUT; no longer R15.1, TP72.1, U19.POUT
- net POUT-PROT: now also R40.2, U7.PA8; no longer R15.2, U4.PA8
- net REG2-PK1: now also C25.1, U12.REG2; no longer C9.1, U2.REG2
- net REG2-PK2: now also C36.1, U17.REG2; no longer C33.1, U15.REG2
- net REG3-PK1: now also C24.1, U12.REG3; no longer C3.1, U2.REG3
- net REG3-PK2: now also C35.1, U17.REG3; no longer C32.1, U15.REG3
- net SWCLK: now also U7.PA14-SWCLK; no longer U4.PA14-SWCLK
- net SWDIO: now also U7.PA13-SWDIO; no longer U4.PA13-SWDIO
- net THRM-PK1: now also R71.2, R73.2, U12.THRM; no longer R41.2, R42.2, U2.THRM
- net THRM-PK2: now also R101.2, R103.2, U17.THRM; no longer R56.2, R57.2, U15.THRM
- net TPS62111-PG1: now also TP12.1; no longer TP79.1
- net TPS62111-SYNC1: now also TP10.1; no longer TP80.1
- net VBATT-F-PK1: now also C19.1, Q10.S, Q20.D, R56.2, R57.2, R63.2, TP37.1, U10.VIN; no longer C30.1, Q1.S, Q14.D, R1.2, R45.2, R70.2, TP6.1, U9.VIN
- net VBATT-F-PK2: now also C30.1, Q28.S, Q31.D, Q38.D, R86.2, R87.2, R93.2, TP60.1, U15.VIN; no longer C28.1, Q28.D, Q29.D, Q32.S, R65.2, R82.2, R90.2, TP61.1, U7.VIN
- net VBATT-PK1: now also C17.1, Q16.D, R54.2, R65.2, TP38.1; no longer C21.1, Q9.D, R39.2, R53.2, TP5.1
- net VBATT-PK2: now also C28.1, Q34.D, R84.2, R95.2, TP61.1; no longer C25.1, Q24.D, R51.2, R60.2, TP60.1
- net VBATT-PL1: now also C20.1, C22.1, R65.1, U12.VBATT; no longer C13.1, C14.1, R39.1, U2.VBATT
- net VBATT-PL2: now also C31.1, C33.1, R95.1, U17.VBATT; no longer C17.1, C22.1, R51.1, U15.VBATT
- net VBUS: now also C23.1, C34.1, Q18.D, Q3.S, Q36.D, TP36.1, TP59.1, U10.SENSE, U11.VIN, U15.SENSE, U16.VIN; no longer C29.1, C31.1, Q15.D, Q18.S, Q27.D, TP62.1, TP7.1, U10.VIN, U7.SENSE, U8.VIN, U9.SENSE
- net VBUSP: now also C6.1, C7.2, Q4.D, R39.2; no longer C38.2, C40.1, Q17.D, R107.2
- net VPD: now also C3.2, R1.2, R15.2, R18.2, R3.2, R9.2, TP1.1, U2.VDD, U3.VDD; no longer C37.2, R109.2, R110.2, R114.2, R118.2, R123.2, TP82.1, U21.VDD, U22.VDD

Commit message: First real thoughts on inhibit switches.
Parts:
- added SW1, SW3: OMRON-D2F-L3-D-LEFT, SW-Omron-D2F-L3-D-switch:OMRON-D2F-L3-D-LEFT
- added SW2, SW4: OMRON-D2F-L3-D-RIGHT, SW-Omron-D2F-L3-D-switch:OMRON-D2F-L3-D-RIGHT
Connections:
- new net N$1: R62.2, SW1.COM, TP43.1, U12.CSN
- net GND: now also SW1.NC; no longer R62.2, TP43.1, U12.CSN
Changed lines of the file:
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@@
 <?xml version="1.0" encoding="utf-8"?>
 <!DOCTYPE eagle SYSTEM "eagle.dtd">
-<eagle version="9.5.1">
+<eagle version="9.6.1">
 <drawing>
 <settings>
@@
 <setting verticaltext="up"/>
 </settings>
-<grid distance="0.1" unitdist="inch" unit="inch" style="lines" multiple="1" display="no" altdistance="0.01" altunitdist="inch" altunit="inch"/>
+<grid distance="0.05" unitdist="inch" unit="inch" style="lines" multiple="2" display="no" altdistance="0.01" altunitdist="inch" altunit="inch"/>
 <layers>
 <layer number="1" name="Top" color="4" fill="1" visible="no" active="no"/>
@@
 <part name="U2" library="U-Microchip-MIC842-Comparator" deviceset="MIC842L" device="YC5"/>
 <part name="U3" library="U-Microchip-MIC842-Comparator" deviceset="MIC842L" device="YC5"/>
+<part name="SW1" library="SW-Omron-D2F-L3-D-switch" deviceset="OMRON-D2F-L3-D" device="-LEFT"/>
+<part name="SW2" library="SW-Omron-D2F-L3-D-switch" deviceset="OMRON-D2F-L3-D" device="-RIGHT"/>
+<part name="SW3" library="SW-Omron-D2F-L3-D-switch" deviceset="OMRON-D2F-L3-D" device="-LEFT"/>
+<part name="SW4" library="SW-Omron-D2F-L3-D-switch" deviceset="OMRON-D2F-L3-D" device="-RIGHT"/>
 </parts>
 <sheets>
@@
 <attribute name="NAME" x="260.35" y="77.978" size="1.778" layer="95" font="vector" align="bottom-center"/>
 </instance>
-<instance part="GND46" gate="1" x="256.54" y="48.26" smashed="yes">
-<attribute name="VALUE" x="254" y="45.72" size="1.778" layer="96"/>
+<instance part="GND46" gate="1" x="259.08" y="30.48" smashed="yes">
+<attribute name="VALUE" x="256.54" y="27.94" size="1.778" layer="96"/>
 </instance>
 <instance part="R65" gate="R" x="294.64" y="148.59" smashed="yes" rot="R180">
@@
 <attribute name="VALUE" x="259.842" y="163.83" size="1.778" layer="96" rot="R90"/>
 </instance>
+<instance part="SW1" gate="G$1" x="256.54" y="40.64" smashed="yes" rot="R270">
+<attribute name="NAME" x="252.73" y="39.37" size="1.778" layer="95" rot="R180"/>
+<attribute name="VALUE" x="252.73" y="41.91" size="1.778" layer="96" rot="R180"/>
+</instance>
+<instance part="SW2" gate="G$1" x="50.8" y="185.42" smashed="yes">
+<attribute name="NAME" x="45.72" y="189.23" size="1.778" layer="95"/>
+<attribute name="VALUE" x="45.72" y="180.34" size="1.778" layer="96"/>
+</instance>
 </instances>
 <busses>
@@
 <net name="GND" class="0">
 <segment>
-<wire x1="346.71" y1="95.25" x2="346.71" y2="58.42" width="0.1524" layer="91"/>
 <pinref part="GND46" gate="1" pin="GND"/>
-<pinref part="R62" gate="R" pin="2"/>
-<wire x1="256.54" y1="50.8" x2="256.54" y2="54.61" width="0.508" layer="91"/>
-<wire x1="256.54" y1="54.61" x2="256.54" y2="58.42" width="0.508" layer="91"/>
-<wire x1="256.54" y1="58.42" x2="346.71" y2="58.42" width="0.1524" layer="91"/>
-<junction x="256.54" y="58.42"/>
-<pinref part="U12" gate="A" pin="CSN"/>
-<pinref part="TP43" gate="G$1" pin="1"/>
-<junction x="256.54" y="54.61"/>
+<wire x1="259.08" y1="33.02" x2="259.08" y2="35.56" width="0.508" layer="91"/>
+<pinref part="SW1" gate="G$1" pin="NC"/>
 </segment>
 <segment>
@@
 </segment>
 </net>
+<net name="N$1" class="0">
+<segment>
+<wire x1="346.71" y1="95.25" x2="346.71" y2="58.42" width="0.1524" layer="91"/>
+<pinref part="R62" gate="R" pin="2"/>
+<wire x1="256.54" y1="45.72" x2="256.54" y2="54.61" width="0.508" layer="91"/>
+<wire x1="256.54" y1="54.61" x2="256.54" y2="58.42" width="0.508" layer="91"/>
+<wire x1="256.54" y1="58.42" x2="346.71" y2="58.42" width="0.1524" layer="91"/>
+<junction x="256.54" y="58.42"/>
+<pinref part="U12" gate="A" pin="CSN"/>
+<pinref part="TP43" gate="G$1" pin="1"/>
+<junction x="256.54" y="54.61"/>
+<pinref part="SW1" gate="G$1" pin="COM"/>
+</segment>
+</net>
 </nets>
 </sheet>
@@
 <attribute name="VALUE" x="260.35" y="162.56" size="1.778" layer="96" rot="R90"/>
 </instance>
+<instance part="SW3" gate="G$1" x="73.66" y="210.82" smashed="yes">
+<attribute name="NAME" x="68.58" y="214.63" size="1.778" layer="95"/>
+<attribute name="VALUE" x="68.58" y="205.74" size="1.778" layer="96"/>
+</instance>
+<instance part="SW4" gate="G$1" x="45.72" y="205.74" smashed="yes">
+<attribute name="NAME" x="40.64" y="209.55" size="1.778" layer="95"/>
+<attribute name="VALUE" x="40.64" y="200.66" size="1.778" layer="96"/>
+</instance>
 </instances>

Commit message: Updated battery card with Oleg's drawings; about to upgrade processors.
Parts:
- removed PCB1: ORESAT-CARD-V1.1-BATTERY, oresat-cards:ORESAT-CARD-V1.1-BATTERY
- removed SW1, SW3: OMRON-D2F-L3-D-LEFT, SW-Omron-D2F-L3-D-switch:OMRON-D2F-L3-D-LEFT
- removed SW2, SW4: OMRON-D2F-L3-D-RIGHT, SW-Omron-D2F-L3-D-switch:OMRON-D2F-L3-D-RIGHT
- added JP10, JP11, JP12, JP5, JP6, JP7, JP8, JP9: (no value), pinhead:PINHD-1X1
- added PCB2: ORESAT-CARD-V1.1-BATTERY-V1.0, oresat-cards:ORESAT-CARD-V1.1-BATTERY-V1.0
Connections:
- new net N$13: JP12.1, R92.1, U17.CSP
- net !SD: now also JP10.1, JP8.1
- net CSP-PK1: now also JP5.1; no longer R62.1, U12.CSP
- net CSP-PK2: now also JP7.1; no longer R92.1, U17.CSP
- net GND: now also JP11.1, JP9.1, R62.2, TP43.1, U12.CSN; no longer SW1.NC
- net N$1: now also JP6.1, R62.1, U12.CSP; no longer R62.2, SW1.COM, TP43.1, U12.CSN
Other:
- note added: "NC Switch"
- note added: "Normally Open inhibit switches (pulls down !SD when pressed)"

Commit message: New F091 processor. Battery layout done! Still needs polishing.
Parts:
- removed C10, C11, C12, C9: 100n, oresat-rcl:C-EU0603-C-NOSILK
- removed C13, C14: 20p, oresat-rcl:C-EU0603-C-NOSILK
- removed D4: GREEN, SparkFun-LED:LED-GREEN0603
- removed J2: ORESAT-DEBUG-CONNECTOR-CARD, oresat-edge_connector:ORESAT-DEBUG-CONNECTOR-CARD
- removed R40, R42: 10k, oresat-rcl:R-US_0603-C-NOSILK
- removed R41: 2.7k, oresat-rcl:R-US_0603-C-NOSILK
- removed R43, R44: 4.7k, oresat-rcl:R-US_0603-C-NOSILK
- removed TP19, TP20, TP21, TP22, TP23, TP24, TP25, TP34: TEST-POINT-LARGE-SQUARE, oresat-misc:TEST-POINT-LARGE-SQUARE
- removed U6: TCAN330, TCAN330:TCAN330
- removed U7: STM32F042K6, STM32F042K:STM32F042K6
- removed X1: 16MHZ-2.5x2mm, low-gain-radio:CRYSTAL-WITH-GND
- added C44, C45, C48, C49, C50: 100n, oresat-rcl:C-EU0603-C-NOSILK
- added C46, C47: 20p, oresat-rcl:C-EU0603-C-NOSILK
- added D10: AMBER, SparkFun-LED:LED-GREEN0603
- added J4: ORESAT-DEBUG-CONNECTOR-SOLAR, oresat-debug-connector:ORESAT-DEBUG-CONNECTOR-SOLAR
- added R110, R112: 10k, oresat-rcl:R-US_0603-C-NOSILK
- added R111, R113, R114: 2.7k, oresat-rcl:R-US_0603-C-NOSILK
- added TP78, TP79, TP80, TP81, TP82, TP83: TEST-POINT, Tova:TEST-POINT
- added U20: TCAN330, TCAN330:TCAN330
- added U21: STM32F091C, U-ST-STM32F091C-uC:STM32F091C
- added X3: 16MHZ-2.5x2mm, low-gain-radio:CRYSTAL-WITH-GND
Connections:
- removed net CAN_SILENT: U6.S, U7.PA9
- removed net CRYSTALIN1: C14.1, U7.PF0-OSC_IN, X1.1
- removed net CRYSTALOUT1: C13.1, U7.PF1-OSC_OUT, X1.2
- removed net N$25: D4.A, R41.1
- removed net N$26: J2.DEBUG-3, TP23.1
- removed net N$27: J2.DEBUG-2, TP22.1
- removed net N$28: J2.DEBUG-1, TP21.1
- removed net N$29: J2.DEBUG-0, TP20.1
- removed net N$30: J2.SWO, TP19.1
- removed net POUT-PROT: R40.2, U7.PA8
- new net CRYSTALIN2: C47.1, U21.PF0-OSC_IN, X3.1
- new net CRYSTALOUT2: C46.1, U21.PF1-OSC_OUT, X3.2
- new net N$101: D10.A, R111.1
- new net N$102: J4.DEBUG-3, TP82.1
- new net N$103: J4.DEBUG-2, TP81.1
- new net N$104: J4.DEBUG-1, TP80.1
- new net N$105: J4.DEBUG-0, TP79.1
- new net N$106: J4.SWO, TP83.1
- new net PA0: R111.2, U21.PA0
- new net PA15: U21.PA15
- new net PA8/POUTPROT: R112.2, U21.PA8
- new net PA9/CAN_SILENT: U20.S, U21.PA9
- new net PB12: U21.PB12
- new net PB13: U21.PB13
- new net PB14: U21.PB14
- new net PB15: U21.PB15
- new net PB3: U21.PB3
- new net PB8: U21.PB8
- new net PB9: U21.PB9
- new net PC13: U21.PC13
- new net PC14: U21.PC14-OSC32_IN
- new net PC15: U21.PC15-OSC32_OUT
- net !SD: no longer TP34.1
- net 3.3V: now also C44.2, C45.2, C48.2, C49.2, C50.2, J4.VTARGET, R113.2, R114.2, U20.VCC, U21.VBAT, U21.VDD, U21.VDDA, U21.VDDIO2; no longer C10.2, C11.2, C12.2, C9.2, J2.VTARGET, R43.2, R44.2, U6.VCC, U7.VDD, U7.VDDA, U7.VDDIO2
- net ALERTA-PK1: now also U21.PB5; no longer U7.PB5
- net ALERTA-PK2: now also U21.PB4; no longer U7.PB1
- net BOOT0: now also R110.2, TP78.1, U21.PF11-BOOT0; no longer R41.2, R42.2, TP24.1, U7.PB8-BOOT0
- net CAN1_H: now also U20.CANH; no longer U6.CANH
- net CAN1_L: now also U20.CANL; no longer U6.CANL
- net CAN_RX: now also U20.RXD, U21.PA11; no longer U6.RXD, U7.PA11
- net CAN_SHDN: now also U20.SHDN, U21.PA10; no longer U6.SHDN, U7.PA10
- net CAN_TX: now also U20.TXD, U21.PA12; no longer U6.TXD, U7.PA12
- net CHARGE-DISABLE-PK1: now also U21.PA4; no longer U7.PA15
- net CHARGE-DISABLE-PK2: now also U21.PB0; no longer U7.PA6
- net CHARGE-STAT-OC-PK1: now also U21.PA7; no longer U7.PA0
- net CHARGE-STAT-OC-PK2: now also U21.PB10; no longer U7.PA4
- net DCHG-STAT-OC-PK1: now also U21.PA1; no longer U7.PA1
- net DCHG-STAT-OC-PK2: now also U21.PB11; no longer U7.PA5
- net DISCHARGE-DISABLE-PK1: now also U21.PA5; no longer U7.PB3
- net DISCHARGE-DISABLE-PK2: now also U21.PB1; no longer U7.PA7
- net FAST-CHARGE-PK1: now also U21.PA6; no longer U7.PB4
- net FAST-CHARGE-PK2: now also U21.PB2; no longer U7.PB0
- net GND: now also C44.1, C45.1, C46.2, C47.2, C48.1, C49.1, C50.1, D10.C, J4.GND, J4.PAD, R110.1, U20.GND, U21.VSS, U21.VSSA, X3.SHIELD; no longer C10.1, C11.1, C12.1, C13.2, C14.2, C9.1, D4.C, J2.GND, J2.PAD, R42.1, U6.GND, U7.VSS, X1.SHIELD
- net NRESET: now also J4.NRST, U21.NRST; no longer J2.NRST, TP25.1, U7.NRST
- net PA2/USART2_TX: now also J4.CARD-TX, U21.PA2; no longer J2.CARD-RX, U7.PA2
- net PA3/USART2_RX: now also J4.CARD-RX, U21.PA3; no longer J2.CARD-TX, U7.PA3
- net PB6/SCL: now also R113.1, U21.PB6; no longer R44.1, U7.PB6
- net PB7/SDA: now also R114.1, U21.PB7; no longer R43.1, U7.PB7
- net POUT: now also R112.1; no longer R40.1
- net SWCLK: now also J4.SWCLK, U21.PA14-SWCLK; no longer J2.SWCLK, U7.PA14-SWCLK
- net SWDIO: now also J4.SWDIO, U21.PA13-SWDIO; no longer J2.SWDIO, U7.PA13-SWDIO
- net VBUS: no longer J2.VBUS
- net VBUSP: now also J4.VBUSP
Other:
- note added: "ALL CAPS 0603 16V X5R 10% OR BETTER"
- note added: "ALL RESISTORS 0603 1% OR BETTER"
- note added: "Each VDD pin bypassed"
- note added: "Power/Current draw from OPD. Signal is analog voltage 0-1.2V"
- note added: "Rx-Tx switch happens on programming board"
- note added: "STM32F09X Microcontroller Design Block"
- note added: "VBAT not bypassed becase not enough room instead tied into nearest bypass cap"
- note removed: "OreSat battery Card - uC"
- note removed: "Power/Current draw from OPD."
- note removed: "Signal is analog voltage 0-1.2V"

Commit message: Some feedback from design review; more text, 100k instead of 10k for some transistors, still missing heaters.
Parts:
- D5, D6, D7, D8: value (none) -> 1N4151W-E3-08
- R113, R114: value 2.7k -> 4.7k
Connections:
- removed net PA15: U21.PA15
- removed net PB12: U21.PB12
- removed net PB13: U21.PB13
- removed net PB14: U21.PB14
- removed net PB15: U21.PB15
- removed net PB3: U21.PB3
- removed net PB8: U21.PB8
- removed net PB9: U21.PB9
- removed net PC13: U21.PC13
- removed net PC14: U21.PC14-OSC32_IN
- removed net PC15: U21.PC15-OSC32_OUT
Other:
- note added: "MOSFETs needed for ground level decoupling."

Commit message: Temporary check in; still need to complete heater circuits.
Parts:
- added D11, D12, D4, D9: 1N4151WS, D-Generic-silicon-SOD-323:DIODE-SOD323-R
- added JP14, JP15, JP16, JP17: (no value), pinhead:PINHD-1X1
- added Q42, Q43: DMP2240UDM, Q-MOSFET-PCH-dual-SOT23-6:MOSFET-PCH-SOT23-6
- added R40, R41, R42, R43: 10k, oresat-rcl:R-US_0603-C-NOSILK
- D5, D6, D7, D8: value 1N4151W-E3-08 -> 1N4151WS; device diode:DIODE-SOD123 -> D-Generic-silicon-SOD-323:DIODE-SOD323-R
- J4: value ORESAT-DEBUG-CONNECTOR-SOLAR -> ORESAT-DEBUG-CONNECTOR-ALL; device oresat-debug-connector:ORESAT-DEBUG-CONNECTOR-SOLAR -> oresat-debug-connector:ORESAT-DEBUG-CONNECTOR-ALL
- R12, R13: value 10k -> 665k
- TP78, TP79, TP80, TP81, TP82, TP83: value TEST-POINT -> TEST-POINT-LARGE-SQUARE; device Tova:TEST-POINT -> oresat-misc:TEST-POINT-LARGE-SQUARE
Connections:
- new net N$18: D11.A, Q43.2.G, R42.2
- new net N$25: D4.A, Q42.2.G, R41.2
- new net N$26: Q42.1.D, Q42.2.S
- new net N$27: Q43.1.D, Q43.2.S
- new net N$28: Q1.1.G, R13.2
- new net N$30: Q1.2.G, R12.2
- new net N$62: D12.A, Q43.1.G, R43.2
- new net N$63: D9.A, Q42.1.G, R40.2
- new net N$64: D11.C, D12.C, D4.C, D9.C
- new net N$92: JP14.1, JP16.1, Q42.2.D, Q43.2.D
- net GND: now also JP15.1, JP17.1; no longer R12.1, R13.1
- net N$47: now also R13.1; no longer Q1.1.G, R13.2
- net N$57: now also R12.1; no longer Q1.2.G, R12.2
- net VBUSP: now also Q42.1.S, Q43.1.S, R40.1, R41.1, R42.1, R43.1
Other:
- note added: "+Y HEATER"
- note added: "-Y HEATER"
- note added: "Add N channel with 2x vote to block"
- note added: "HEATER"
- note added: "If it's really vbusp, we need to increase the current in the CB"
- moved on the sheet: C48, D10, R111, R112, R12, R13, U20
