File: eagle/oresat-batteries-prototype.brd (EAGLE design)
At the start: 42 x 63 mm, 81 parts, among them Q10 BSS84, Q11 BSS84, Q12 Si7625DN, Q13 Si7625DN, Q14 Si7625DN, Q15 Si7625DN, Q16 Si7625DN, Q2 Si7625DN, Q9 Si7625DN, U10 LTC4412, U11 S-8209AAA-T8T1U, U12 S-8209AAA-T8T1U, U2 MAX17205G, U9 LTC4412

Commit message: v1.0 of the battery pack prototype board
Parts:
- removed T1, T2, T3, T4, T5, T6: (no value), zetex:SOT-23
- added Q1, Q3, Q4, Q5, Q6, Q7: PMV45EN, Tova:SOT23
- added TP1, TP3, TP4, TP5: TEST-POINT, Tova:2MM-TEST-POINT
- Q10, Q11: value BSS84 -> NTR4101P; device Transistor:SOT23 -> Tova:SOT23
- moved R66 0.56 mm to (15.2, 16.0)
- moved R74 0.06 mm to (9.30, 47.3)
Connections:
- net !FAST-CHARGE-PK1: now also Q1.3; no longer T2.1
- net CHARGE-DISABLE: now also Q6.1; no longer T6.3
- net CSP-PK1: now also Q3.2, Q4.2, Q5.2, Q6.2, Q7.2, TP3.1; no longer T1.2, T3.2, T4.2, T5.2, T6.2
- net DISCHARGE-DISABLE: now also Q7.1; no longer T5.3
- net FAST-CHARGE-PK1: now also Q1.1; no longer T2.3
- net GND: now also Q1.2; no longer T2.2
- net N$1: now also Q5.3; no longer T4.1
- net N$10: now also Q3.3; no longer T3.1
- net N$11: now also Q4.1, Q7.3; no longer T1.3, T5.1
- net N$42: now also TP4.1
- net N$5: now also Q4.3; no longer T1.1
- net N$51: now also Q3.1, Q6.3; no longer T3.3, T6.1
- net N$53: now also TP1.1
- net N$54: now also TP5.1
- net OPD-PK1-DISABLE: now also Q5.1; no longer T4.3
Routing:
- net N$53: track 11.3 -> 14.5 mm
- net N$42: track 11.4 -> 14.5 mm
- net VBATT-PK1: track 27.6 -> 29.2 mm
- net GND: vias 6 -> 50
Other:
- board text added: "!SD"
- board text added: "+ CELL 1"
- board text added: "+ CELL 2"
- board text added: "- CELL 1"
- board text added: "- CELL 2"
- board text added: "ALERT"
- board text added: "CDIS"
- board text added: "CSTAT"
- board text added: "DDIS"
- board text added: "DSTAT"
- board text added: "FASTCHG"
- board text added: "GND"
- board text added: "PACK +"
- board text added: "PACK -"
- board text added: "PKDIS"
- board text added: "SCL"
- board text added: "SDA"
- board text added: "THERM Cell 1"
- board text added: "THERM Cell 2"
