File: kicad/oresat-batteries-sch-mcu.kicad_sch (KiCad schematic)
At the start: 51 parts, among them J4 ORESAT-DEBUG-CONNECTOR-ALL, Q20 PMV45EN, Q21 PMV45EN, Q38 PMV45EN, Q39 PMV45EN, Q42 MOSFET-PCH-SOT23-6, Q43 MOSFET-PCH-SOT23-6, U20 TCAN330, U21 STM32F091C, X3 CRYSTAL-WITH-GND

Commit message: Updating KiCAD import of EAGLE battery card v3.0 and calling it v3.1 because the gerber files will definitely be different and we'll probably implement a few small changes. Reimports, renames, and fixes .gitignore file. Oh and makes the worksheets pretty.
Other:
- note removed: "1.0"
- note removed: "ALL CAPS 0603 16V X5R 10% OR BETTER"
- note removed: "ALL RESISTORS 0603 1% OR BETTER"
- note removed: "STM32F09X Microcontroller Design Block"
- title: (none) -> OreSat Battery Card - Microcontroller
- moved on the sheet: C44, C45, C46, C47, C48, C49, C50, D10, D11, D12, D4, D9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
