File: kicad/oresat-batteries-sch-pack-2.kicad_sch (KiCad schematic)
At the start: 85 parts, among them Q11 SI7111EDN-T1-GE3, Q22 SQS484ENW-T1_GE3, Q24 PMV45ENR, Q25 PMV45ENR, Q26 PMV45ENR, Q27 PMV45ENR, Q30 SI7111EDN-T1-GE3, Q31 SI7111EDN-T1-GE3, Q32 NTR4101, Q33 NTR4101, Q34 SI7111EDN-T1-GE3, Q35 SI7111EDN-T1-GE3, Q36 SI7111EDN-T1-GE3, Q37 SI7111EDN-T1-GE3, U13 S-8209AAA-T8T1U, U14 S-8209AAA-T8T1U, U15 LTC4412, U16 LTC4412, U17 MAX17205G

Commit message: Not sure what changed from back in February, but committing anyway :)
Parts:
- added RT3, RT4: 10k NTC TH, symbol Device:Thermistor
- C11: DIS Digi-Key -> DigiKey; DPN 1276-2893-1-ND -> 490-GRT21BC71E106KE13KCT-ND; MFR Samsung -> Murata Electronics; MPN CL21A106KOFNNNE -> GRT21BC71E106KE13K
- C26, C28, C30, C33, C34: DIS Digi-Key -> DigiKey; DPN 399-1099-1-ND -> 399-6856-1-ND; MFR Kemet -> KEMET; MPN C0603C104M4RACTU -> C0603C104K5RACAUTO
- C27, C29: DIS (none) -> DigiKey; DPN 399-7842-1-ND -> 399-12983-1-ND; MFR Kemet -> KEMET; MPN C0603C103M5RACTU -> C0603C103J5RACAUTO
- C31, C32: DIS Digi-Key -> DigiKey; DPN 311-1080-1-ND -> 399-12989-1-ND; MFR Yageo -> KEMET; MPN CC0603KRX7R9BB102 -> C0603C102J5RACAUTO
- C35, C36: DIS Digi-Key -> DigiKey; DPN 399-7934-1-ND -> 399-6820-1-ND; MFR Kemet -> KEMET; MPN C0603C474K4PACTU -> C0603C473K5RACAUTO
- D13, D7, D8: DIS (none) -> DigiKey; DPN (none) -> 112-1N4151WS-E3-08CT-ND; MFR (none) -> Vishay; MPN (none) -> 1N4151WS-E3-08
- F2: DIS (none) -> DigiKey; DPN (none) -> 18-1206L500/12SLPRCT-ND; MFR (none) -> Littelfuse Inc; MPN (none) -> 18-1206L500/12SLPRCT-ND
- F4: DIS (none) -> DigiKey; DPN (none) -> F5765CT-ND; MFR (none) -> Littelfuse Inc; MPN (none) -> F5765CT-ND
- JP3, JP4: DIS (none) -> N/A; DPN (none) -> N/A; MFR (none) -> N/A; MPN (none) -> N/A; now left out of the parts list
- Q11, Q30, Q31, Q34, Q35, Q36, Q37: DPN SI7625DN-T1-GE3CT-ND -> SI7111EDN-T1-GE3CT-ND; MPN SI7625DN-T1-GE3 -> SI7111EDN-T1-GE3
- Q22: DPN (none) -> SQS484ENW-T1_GE3CT-ND; MFR (none) -> Vishay; MPN (none) -> SQS484ENW-T1_GE3
- R101, R103: DIS Digi-Key -> DigiKey; DPN 311-10.0KHRCT-ND -> RMCF0603FT10K0CT-ND; MFR Yageo -> Stackpole Electronics; MPN RC0603FR-0710KL -> RMCF0603FT10K0
- R56, R97: DIS Digi-Key -> DigiKey; DPN RR08P100KDCT-ND -> RMCF0603FT100KCT-ND; MFR Yageo -> Stackpole Electronics; MPN RR0816P-104-D -> RMCF0603FT100K
- R70: DIS Digi-Key -> DigiKey; DPN RR08P100KDCT-ND -> RMCF0603FT100KCT-ND; MFR Susumu -> Stackpole Electronics; MPN RR0816P-104-D -> RMCF0603FT100K
- R75, R78, R82, R83: DIS Digi-Key -> DigiKey; DPN 311-1.0KGRCT-ND -> RMCF0603FT2K70CT-ND; MFR Yageo -> Stackpole Electronics; MPN RC0603JR-071KL -> RMCF0603FT1K00
- R76, R79, R86, R88, R89, R90, R91: DIS Digi-Key -> DigiKey; DPN 311-1.00MHRCT-ND -> RMCF0603FT100KCT-ND; MFR Yageo -> Stackpole Electronics; MPN RC0603FR-071ML -> RMCF0603FT100K
- R77, R80: DIS Digi-Key -> DigiKey; DPN 311-10.0KHRCT-ND -> RMCF0603FT100KCT-ND; MFR Yageo -> Stackpole Electronics; MPN RC0603FR-0710KL -> RMCF0603FT100K
- R81, R84: DIS Digi-Key -> DigiKey; DPN 311-470GRCT-ND -> RMCF0603FT470RCT-ND; MFR Yageo -> Stackpole Electronics; MPN RC0603JR-07470RL -> RMCF0603FT470R
- R92: DIS Digi-Key -> DigiKey
- R94: DIS Digi-Key -> DigiKey; DPN RR08P4.7KDCT-ND -> RMCF0603FT10K0CT-ND; MFR TE Connectivity -> Stackpole Electronics; MPN RR0816P-472-D -> RMCF0603FT10K0
- R95: DPN 311-10.0HRCT-ND -> RMCF0603FT10R0CT-ND; MFR Yageo -> Stackpole Electronics; MPN RC0603FR-0710RL -> RMCF0603FT10R0
- R96: DPN 311-100HRCT-ND -> RMCF0603FT100RCT-ND; MFR Yageo -> Stackpole Electronics; MPN RC0603FR-07100RL -> RMCF0603FT100R
- U13, U14: DIS (none) -> Mouser; DPN (none) -> 628-S-8209AAA-T8T1U
- U15, U16: DIS Digi-Key -> DigiKey; DPN LTC4412ES6#TRPBFCT-ND -> MAX4211FETE+-ND; MPN LTC4412ES6#TRPBF -> MAX4211FETE
- U17: MPN MAX17205G+T -> MAX17205G
Connections:
- no-connect marks 3 -> 7

Commit message: Updated data, spiffed up the root page, renamed some STM specific OPD signals, synced SCH and BRD, fixed a bunch of DRC errors, NOW ready for MCXN import that will screw everything up.
Changed lines of the file:
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@@
 	(title_block
 		(title "OreSat Battery Card")
-		(date "2026-01-10")
+		(date "2026-03-23")
 		(rev "4.0")
 		(company "Portland State Aerospace Society")
@@
 		)
 	)
-	(wire
-		(pts
-			(xy 278.13 45.72) (xy 278.13 44.45)
-		)
-		(stroke
-			(width 0.1524)
-			(type solid)
-		)
-	)
 	(polyline
 		(pts
@@
 	(wire
 		(pts
-			(xy 278.13 60.96) (xy 278.13 59.69)
-		)
-		(stroke
-			(width 0)
-			(type default)
-		)
-	)
-	(wire
-		(pts
 			(xy 58.42 175.26) (xy 58.42 171.45)
 		)
@@
 		)
 		(instances
-			(project ""
+			(project "oresat-batteries"
 				(path "/d5070776-2522-4f7b-9d31-10770161e48a/714b8cb1-7fa6-448b-9eed-93330aa30436"
 					(reference "RT3")
@@
 		)
 		(instances
-			(project ""
+			(project "oresat-batteries"
 				(path "/d5070776-2522-4f7b-9d31-10770161e48a/714b8cb1-7fa6-448b-9eed-93330aa30436"
 					(reference "RT4")
