File: kicad/oresat-batteries.kicad_pcb (KiCad board)
At the start: 4 copper layers, 99.8 x 94.6 mm, 318 parts, among them J1 J-SAMTEC-TFM-120-X1-XXX-D-RA, J2 SM14B-SHLS-TF, Q1 DMP2240UDM-7, Q10 SI7111EDN-T1-GE3, Q11 SI7111EDN-T1-GE3, Q12 SI7111EDN-T1-GE3, Q13 SI7111EDN-T1-GE3, Q14 NTR4101, Q15 NTR4101, Q16 SI7111EDN-T1-GE3, Q17 SI7111EDN-T1-GE3, Q18 SI7111EDN-T1-GE3, Q19 SI7111EDN-T1-GE3, Q2 PMV45ENR, Q20 PMV45ENR, Q21 PMV45ENR, Q22 SQS484ENW-T1_GE3, Q24 PMV45ENR, Q25 PMV45ENR, Q26 PMV45ENR, Q27 PMV45ENR, Q29 SQS484ENW-T1_GE3, Q3 DMP3050LVTQ-7, Q30 SI7111EDN-T1-GE3, Q31 SI7111EDN-T1-GE3, Q32 NTR4101, Q33 NTR4101, Q34 SI7111EDN-T1-GE3, Q35 SI7111EDN-T1-GE3, Q36 SI7111EDN-T1-GE3, Q37 SI7111EDN-T1-GE3, Q38 PMV45ENR, Q39 PMV45ENR, Q4 DMP3050LVTQ-7, Q42 DMP2240UDM-7, Q43 DMP2240UDM-7, Q44 PMV45ENR, Q5 PMV45ENR, Q6 PMV45ENR, Q7 PMV45ENR, Q8 PMV45ENR, Q9 PMV45ENR, SW1 Omron D2F-L3-D (LEFT), SW2 Omron D2F-L3-D (RIGHT), SW3 OMRON D2F-L3-D (LEFT), SW4 OMRON D2F-L3-D (RIGHT), U1 MAX7310, U10 LTC4412, U11 LTC4412, U12 MAX17205G, U13 S-8209AAA-T8T1U, U14 S-8209AAA-T8T1U, U15 LTC4412, U16 LTC4412, U17 MAX17205G, U2 MIC842LYC5, U20 TCAN330, U21 STM32F091C, U3 MIC842LYC5, U4 MAX4211, U5 TPS62111RSA, U6 TS5A21366DCUR, U8 S-8209AAA-T8T1U, U9 S-8209AAA-T8T1U, X3 ECS-160-10-36Q-ES-TR

Commit message: Not sure what changed from back in February, but committing anyway :)
Parts:
- R11, R17, R5: value 1K -> 1k
- R29: value NP -> 10k
- SW1: value Omron D2F-L3-D (LEFT) -> D2F-L3-D (LEFT)
- SW2: value Omron D2F-L3-D (RIGHT) -> D2F-L3-D (RIGHT)
- SW3: value OMRON D2F-L3-D (LEFT) -> D2F-L3-D (LEFT)
- SW4: value OMRON D2F-L3-D (RIGHT) -> D2F-L3-D (RIGHT)
- U20: value TCAN330 -> TCAN330G

Commit message: Updated data, spiffed up the root page, renamed some STM specific OPD signals, synced SCH and BRD, fixed a bunch of DRC errors, NOW ready for MCXN import that will screw everything up.
Parts:
- removed TP4, TP6, TP7: TEST-POINT-LARGE-SQUARE, oresat-misc:TestPoint-0.75mm-th
- D1: value GRN -> AMB
- R10, R14, R15, R16, R2, R29, R3, R35, R4, R8, R9: footprint oresat-batteries:.0603-C-NOSILK -> oresat-passives:0603-C-NOSILK
- R57, R67: value 10k -> 1k
- moved TP2 1.20 mm to (137.5, 71.2)
- moved U3 0.36 mm to (137.2, 75.0)
- moved U2 0.20 mm to (139.9, 68.5)
- moved R12 0.16 mm to (137.2, 68.8), turned to -90 degrees
Connections:
- net /Battery Pack 1 (BOTTOM)/PB6/SCL renamed /Battery Pack 1 (BOTTOM)/I2C1_SCL
- net /Battery Pack 1 (BOTTOM)/PB7/SDA renamed /Battery Pack 1 (BOTTOM)/I2C1_SDA
- net /Microcontroller/PA2/USART2_TX renamed /Microcontroller/MCU-UART-TX
- net /Microcontroller/PA3/USART2_RX renamed /Microcontroller/MCU-UART-RX
- net /Power/AD0 renamed /OreSat Power Domain (OPD)/AD0
- net /Power/AD1 renamed /OreSat Power Domain (OPD)/AD1
- net /Power/AD2 renamed /OreSat Power Domain (OPD)/AD2
- net /Power/CB-RESET renamed /OreSat Power Domain (OPD)/CB-RESET
- net /Power/CB_CTRL renamed /OreSat Power Domain (OPD)/CB_CTRL
- net /Power/PEN-SCL-FILT renamed /OreSat Power Domain (OPD)/PEN-SCL-FILT
- net /Power/PEN-SDA-FILT renamed /OreSat Power Domain (OPD)/PEN-SDA-FILT
- net /Power/UART_EN renamed /OreSat Power Domain (OPD)/UART_EN
- net /Power/~{FAULT} renamed /OreSat Power Domain (OPD)/~{FAULT}
- C4 pad 1: /Power/ON/~{OFF} -> /OreSat Power Domain (OPD)/ON/~{OFF}
- C9 pad 2: VPD -> /OreSat Power Domain (OPD)/ON/~{OFF}
- Q2 pad 1: /Power/ON/~{OFF} -> /OreSat Power Domain (OPD)/ON/~{OFF}
- R23 pad 2: /Power/ON/~{OFF} -> /OreSat Power Domain (OPD)/ON/~{OFF}
- R24 pad 2: /Power/ON/~{OFF} -> /OreSat Power Domain (OPD)/ON/~{OFF}
- TP8 pad 1: /Power/ON/~{OFF} -> /OreSat Power Domain (OPD)/ON/~{OFF}
- U1 pad 8: /Power/ON/~{OFF} -> /OreSat Power Domain (OPD)/ON/~{OFF}
- U4 pad 1: /Power/ON/~{OFF} -> /OreSat Power Domain (OPD)/ON/~{OFF}
- U6 pad 8: VPD -> /OreSat Power Domain (OPD)/ON/~{OFF}
Routing:
- net /OreSat Power Domain (OPD)/ON/~{OFF}: track 0.00 -> 80.7 mm, vias 0 -> 3
- net /Power/ON/~{OFF}: track 55.3 -> 0.00 mm, vias 2 -> 0
- net VPD: track 75.8 -> 71.2 mm, vias 7 -> 6
- net Net-(U3-OUT): track 5.16 -> 2.00 mm
- net Net-(U2-OUT): track 4.96 -> 1.87 mm, vias 1 -> 0
- net GND: track 28.3 -> 30.1 mm
- net Net-(Q1B-G): track 1.22 -> 2.37 mm
- net Net-(U8-VDD): track 5.98 -> 6.99 mm
- net VBUSP: track 129.2 -> 128.5 mm, vias 14 -> 12
- net /OreSat Power Domain (OPD)/PEN-SCL-FILT: track 31.8 -> 31.1 mm
- net Net-(Q2-D): vias 1 -> 0
- net /Battery Pack 2 (TOP)/BATTNEG-PK2: vias 4 -> 3
