File: kicad/oresat-batteries-sch-pack-1.kicad_sch (KiCad schematic)
At the start: 87 parts, among them Q10 SI7111EDN-T1-GE3, Q12 SI7111EDN-T1-GE3, Q13 SI7111EDN-T1-GE3, Q14 NTR4101, Q15 NTR4101, Q16 SI7111EDN-T1-GE3, Q17 SI7111EDN-T1-GE3, Q18 SI7111EDN-T1-GE3, Q19 SI7111EDN-T1-GE3, Q29 SQS484ENW-T1_GE3, Q6 PMV45ENR, Q7 PMV45ENR, Q8 PMV45ENR, Q9 PMV45ENR, U10 LTC4412, U11 LTC4412, U12 MAX17205G, U8 S-8209AAA-T8T1U, U9 S-8209AAA-T8T1U

Commit message: Intermediary state on v4. Added one of two efuses.
Parts:
- removed F1: 1206L500/12SLPR, oresat-passives:1206-C, symbol Device:Polyfuse_Small
- removed Q12: SI7111EDN-T1-GE3, Package_SO:Vishay_PowerPAK_1212-8_Single, symbol Transistor_FET:SiS443DN
- removed U10: LTC4412, Package_TO_SOT_SMD:TSOT-23-6, symbol Power_Management:LTC4412xS6
- added C46, C47, C49: 100n, oresat-passives:0603-C-NOSILK, symbol Device:C_Small
- added Q23: DMP2035UQ-7, Package_TO_SOT_SMD:SOT-23, symbol Transistor_FET:Q_PMOS_GSD
- added R104, R107, R109, R68: 100k, oresat-passives:0603-C-NOSILK, symbol Device:R_Small_US
- added R72: 1870, oresat-passives:0603-C-NOSILK, symbol Device:R_Small_US
- added U10: TPS25983, oresat-ics:U-TPS259830LNRGER, symbol oresat-ics:TPS25983
- B1, B2: value B-18650-LI-BATTERY -> Tenergy 30005; symbol oresat-batteries-eagle-import:B-18650-LI-BATTERY -> Device:Battery_Cell
- C19: value 100n -> 15n
- Q14, Q15: value NTR4101 -> DMP2035UQ-7; DPN NTR4101PT1GOSCT-ND -> 31-DMP2035UQ-7CT-ND; MFR ON Semi -> Diodes Incorporated; MPN NTR4101PT1G -> DMP2035UQ-7
- Q6, Q7, Q8, Q9: value PMV45ENR -> DMN2053UQ-13; DPN 1727-2307-1-ND -> 31-DMN2053UQ-13CT-ND; MFR Nexperia -> Diodes Incorporated; MPN PMV45EN2R -> DMN2053UQ-13
- R74: value 100k -> 210
Connections:
- net DCHG-STAT-OC-PK1: now also U10.13 (PG)
- net GND: now also R74.2, C46.2, C47.2, C49.2, R104.1, R72.2, U10.11 (NRETRY), U10.12 (OVLO), U10.[4,5,14,26] (GND)
- net VBATT-PK1: now also C49.1, Q23.2 (S), R109.1, U10.[1-3,16,25] (IN)
- net ~{DISCHARGE-PK1}: now also Q23.1 (G), R109.2; no longer R74.2
- net at Q13.5 (D), TP23.1: now also U10.[17-24] (OUT); no longer C19.1
- net at Q13.4 (G): now also R68.1
- net at R74.1: now also U10.8 (ILIM)
- new net: C19.1, R68.2, U10.15 (DVDT/BGATE)
- new net: C47.1, U10.10 (RETRY_DLY)
- new net: Q23.3 (D), R107.2
- new net: R104.2, R107.1, U10.6 (EN/UVLO)
- new net: C46.1, U10.7 (ITIMER)
- new net: R72.1, U10.9 (IMON)
Other:
- note added: "EFUSE Current limit: 7.1 A Voltage ramp up time: 24 ms Transient overcurrent timer: 2.0 ms Time between retries: 4.6 s"
- note added: "Retry every 4.7 s"
- note added: "Retry indefinitely"
- note removed: "PTC @ 5A"
- moved on the sheet: C19, D5, D6, R54, TP23, TP27, TP32, TP33, TP35

Commit message: Schematic complete with new TPS circuit breaker; layout in progress
Parts:
- removed TP27, TP29: TEST-POINT-LARGE-SQUARE, oresat-misc:TestPoint-0.75mm-th, symbol oresat-misc:Test-Point-0.75mm-th
Other:
- note added: "Cell UVLO/OVLO Control"
- note added: "Charge Control"
- note added: "Discharge Control"
- note added: "Off board on leads, thermally connected to battery cells"
- note removed: "CHARGE SWITCH"
- moved on the sheet: B1, B2, C10, C15, C16, C17, C18, C19, C20, C21, C22, C23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
