File: oresat-battery-card/oresat-batteries-sch-heater.kicad_sch (KiCad schematic)
At the start: 22 parts, among them Q20 DMN2053UQ-13, Q21 DMN2053UQ-13, Q38 DMN2053UQ-13, Q39 DMN2053UQ-13, Q42 DMP2240UDM-7, Q43 DMP2240UDM-7

Commit message: Jumped back on the TPS bandwagon - LCSC to the rescue! - and lots of cleanup.
Parts:
- JP14, JP15, JP16, JP17: now not fitted
Other:
- note added: "Diodes prevent gate ruptures from any single P Ch MOSFET from turning on all P CH MOSFETs"
- note removed: "Diodes prevent gate ruptures to heater from turning on all P CH MOSFETs"
Changed lines of the file:
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@@
 	(title_block
 		(title "OreSat Battery Card")
-		(date "2026-03-23")
+		(date "2026-09-27")
 		(rev "4.0")
 		(company "Portland State Aerospace Society")
@@
 		)
 	)
-	(text "Diodes prevent gate ruptures to heater \nfrom turning on all P CH MOSFETs"
+	(text "Diodes prevent gate ruptures from any single\nP Ch MOSFET from turning on all P CH MOSFETs"
 		(exclude_from_sim no)
-		(at 193.548 120.142 0)
+		(at 190.246 121.158 0)
 		(effects
 			(font
@@
 		(on_board yes)
 		(in_pos_files yes)
-		(dnp no)
+		(dnp yes)
 		(property "Reference" "JP17"
 			(at 285.496 144.526 0)
@@
 		(on_board yes)
 		(in_pos_files yes)
-		(dnp no)
+		(dnp yes)
 		(property "Reference" "JP14"
 			(at 268.224 136.652 0)
@@
 		(on_board yes)
 		(in_pos_files yes)
-		(dnp no)
+		(dnp yes)
 		(property "Reference" "JP16"
 			(at 285.242 136.906 0)
@@
 		(on_board yes)
 		(in_pos_files yes)
-		(dnp no)
+		(dnp yes)
 		(property "Reference" "JP15"
 			(at 268.478 144.272 0)

Commit message: Changes to eFuse after trying evaluation board, and recalculating values, and trying to reduce number of passive components to minimum number
Other:
- note added: "At 8.2V and 24.5 ohms, we should see a maximum of ~ 335 mA of current through the heaters."
- note removed: "At 8.2V and 24.5 ohms, we should see a maximum of ~ 343 mA"
Changed lines of the file:
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@@
 		)
 	)
-	(text "At 8.2V and 24.5 ohms, we should see a maximum of ~ 343 mA"
+	(text "At 8.2V and 24.5 ohms, we should see a maximum \nof ~ 335 mA of current through the heaters."
 		(exclude_from_sim no)
-		(at 277.114 172.212 0)
+		(at 277.114 172.974 0)
 		(effects
 			(font
