File: oresat-battery-card/oresat-batteries.kicad_pcb (KiCad board)
At the start: 4 copper layers, 99.8 x 94.6 mm, 345 parts, among them J1 TFM-120-01-L-D-RA, J2 SM14B-SHLS-TF, Q1 DMP2240UDM-7, Q13 SI7111EDN-T1-GE3, Q14 DMP2035UQ-7, Q15 DMP2035UQ-7, Q16 SI7111EDN-T1-GE3, Q17 SI7111EDN-T1-GE3, Q18 SI7111EDN-T1-GE3, Q19 SI7111EDN-T1-GE3, Q2 DMN2053UQ-13, Q20 DMN2053UQ-13, Q21 DMN2053UQ-13, Q22 SQS484ENW-T1_GE3, Q23 DMP2035UQ-7, Q24 DMN2053UQ-13, Q25 DMN2053UQ-13, Q26 DMN2053UQ-13, Q27 DMN2053UQ-13, Q29 SQS484ENW-T1_GE3, Q3 DMP3050LVTQ-7, Q31 SI7111EDN-T1-GE3, Q32 DMP2035UQ-7, Q33 DMP2035UQ-7, Q34 SI7111EDN-T1-GE3, Q35 SI7111EDN-T1-GE3, Q36 SI7111EDN-T1-GE3, Q37 SI7111EDN-T1-GE3, Q38 DMN2053UQ-13, Q39 DMN2053UQ-13, Q4 DMP3050LVTQ-7, Q40 DMP2035UQ-7, Q42 DMP2240UDM-7, Q43 DMP2240UDM-7, Q44 DMN2053UQ-13, Q5 DMN2053UQ-13, Q6 DMN2053UQ-13, Q7 DMN2053UQ-13, Q8 DMN2053UQ-13, Q9 DMN2053UQ-13, SW1 D2F-L3-D3 (LEFT), SW2 D2F-L3-D3 (RIGHT), SW3 D2F-L3-D3 (LEFT), SW4 D2F-L3-D3 (RIGHT), U1 MAX7310, U10 TPS259830ONRGER, U11 LTC4412, U12 MAX17205G, U13 S-8209AAA-T8T1U, U14 S-8209AAA-T8T1U, U15 TPS259830ONRGER, U16 LTC4412, U17 MAX17205G, U2 MIC842LYC5, U20 TCAN337G, U3 MIC842LYC5, U4 MAX4211, U5 TPS62111RSA, U6 TS5A21366DCUR, U7 MCXN947VKLT, U8 S-8209AAA-T8T1U, U9 S-8209AAA-T8T1U, Y2 24 MHz

Commit message: Added imon capabilities, cleaned up some lingering DRCs that kept popping back up.
Parts:
- removed TP34: TEST-POINT-LARGE-SQUARE, oresat-misc:TestPoint-0.75mm-th
- added C67: 100n, oresat-passives:0603-C-NOSILK, F.Cu at (168.2, 103.0)
- added C68: 100n, oresat-passives:0603-C-NOSILK, F.Cu at (170.5, 63.2)
- added R120: 10k, oresat-passives:0603-C-NOSILK, F.Cu at (168.2, 104.2)
- added R121: 10k, oresat-passives:0603-C-NOSILK, F.Cu at (170.5, 64.3)
- C16, C18, C27, C29: value 10n -> 15n
- C46, C61: value 100n -> 15n
- R107, R116: value 357k -> 330k
- R112, R72: value 1k -> 470
- R34: value 20k -> 10k
Connections:
- U7 pad 50: /Microcontroller/P5_2 -> /Battery Pack 1 (BOTTOM)/IMON-PK1
- U7 pad 51: /Microcontroller/P5_3 -> /Battery Pack 2 (TOP)/IMON-PK2
Routing:
- net /Battery Pack 2 (TOP)/IMON-PK2: track 0.00 -> 54.5 mm, vias 0 -> 2
- net /Battery Pack 1 (BOTTOM)/IMON-PK1: track 0.00 -> 31.2 mm, vias 0 -> 2
- net Net-(U15-IMON): track 5.19 -> 7.62 mm
- net /Microcontroller/P5_3: track 1.37 -> 0.00 mm
- net Net-(U10-IMON): track 7.33 -> 8.51 mm
- net /Battery Pack 2 (TOP)/INTERCELL-PK2: track 131.8 -> 132.5 mm
- net Net-(JP3-Pin_1): track 54.6 -> 54.0 mm
- net /Microcontroller/MOARPWR: vias 2 -> 4
