File: oresat-battery-card/oresat-batteries.kicad_pcb (KiCad board)
At the start: 4 copper layers, 99.8 x 94.6 mm, 348 parts, among them J1 TFM-120-01-L-D-RA, J2 SM14B-SHLS-TF, Q1 DMP2240UDM-7, Q13 SI7111EDN-T1-GE3, Q14 DMP2035UQ-7, Q15 DMP2035UQ-7, Q16 SI7111EDN-T1-GE3, Q17 SI7111EDN-T1-GE3, Q18 SI7111EDN-T1-GE3, Q19 SI7111EDN-T1-GE3, Q2 DMN2053UQ-13, Q20 DMN2053UQ-13, Q21 DMN2053UQ-13, Q22 SQS484ENW-T1_GE3, Q23 DMP2035UQ-7, Q24 DMN2053UQ-13, Q25 DMN2053UQ-13, Q26 DMN2053UQ-13, Q27 DMN2053UQ-13, Q29 SQS484ENW-T1_GE3, Q3 DMP3050LVTQ-7, Q31 SI7111EDN-T1-GE3, Q32 DMP2035UQ-7, Q33 DMP2035UQ-7, Q34 SI7111EDN-T1-GE3, Q35 SI7111EDN-T1-GE3, Q36 SI7111EDN-T1-GE3, Q37 SI7111EDN-T1-GE3, Q38 DMN2053UQ-13, Q39 DMN2053UQ-13, Q4 DMP3050LVTQ-7, Q40 DMP2035UQ-7, Q42 DMP2240UDM-7, Q43 DMP2240UDM-7, Q44 DMN2053UQ-13, Q5 DMN2053UQ-13, Q6 DMN2053UQ-13, Q7 DMN2053UQ-13, Q8 DMN2053UQ-13, Q9 DMN2053UQ-13, SW1 D2F-L3-D3 (LEFT), SW2 D2F-L3-D3 (RIGHT), SW3 D2F-L3-D3 (LEFT), SW4 D2F-L3-D3 (RIGHT), U1 MAX7310, U10 TPS259830ONRGER, U11 LTC4412, U12 MAX17205G, U13 S-8209AAA-T8T1U, U14 S-8209AAA-T8T1U, U15 TPS259830ONRGER, U16 LTC4412, U17 MAX17205G, U2 MIC842LYC5, U20 TCAN337G, U3 MIC842LYC5, U4 MAX4211, U5 TPS62111RSA, U6 TS5A21366DCUR, U7 MCXN947VKLT, U8 S-8209AAA-T8T1U, U9 S-8209AAA-T8T1U, Y2 24 MHz

Commit message: Fix CAN trasnceiver part number
Parts:
- U20: value TCAN337G -> TCAN337GDCN
Changed lines of the file:
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@@
 			)
 		)
-		(property "Datasheet" "https://search.kemet.com/download/specsheet/C0603C473K5RACAUTO"
+		(property "Datasheet" "https://www.yageogroup.com/content/datasheet/asset/file/KEM_C1023_X7R_AUTO_SMD"
 			(at 0 0 0)
 			(layer "F.Fab")
@@
 			)
 		)
-		(property "Description" "0.047 µF ±10% 50V Ceramic Capacitor X7R 0603 (1608 Metric)"
+		(property "Description" "0.47 µF ±10% 25V Ceramic Capacitor X7R 0603 (1608 Metric)"
 			(at 0 0 0)
 			(layer "F.Fab")
@@
 			)
 		)
-		(property "DPN" "399-6820-1-ND"
+		(property "DPN" "399-C0603C474K3RACAUTOCT-ND"
 			(at 0 0 0)
 			(unlocked yes)
@@
 			)
 		)
-		(property "MPN" "C0603C473K5RACAUTO"
+		(property "MPN" "C0603C474K3RACAUTO"
 			(at 0 0 0)
 			(unlocked yes)
@@
 			)
 		)
-		(property "Datasheet" "https://search.kemet.com/download/specsheet/C0603C473K5RACAUTO"
+		(property "Datasheet" "https://www.yageogroup.com/content/datasheet/asset/file/KEM_C1023_X7R_AUTO_SMD"
 			(at 0 0 270)
 			(layer "F.Fab")
@@
 			)
 		)
-		(property "Description" "0.047 µF ±10% 50V Ceramic Capacitor X7R 0603 (1608 Metric)"
+		(property "Description" "0.47 µF ±10% 25V Ceramic Capacitor X7R 0603 (1608 Metric)"
 			(at 0 0 270)
 			(layer "F.Fab")
@@
 			)
 		)
-		(property "DPN" "399-6820-1-ND"
+		(property "DPN" "399-C0603C474K3RACAUTOCT-ND"
 			(at 0 0 270)
 			(unlocked yes)
@@
 			)
 		)
-		(property "MPN" "C0603C473K5RACAUTO"
+		(property "MPN" "C0603C474K3RACAUTO"
 			(at 0 0 270)
 			(unlocked yes)
@@
 			)
 		)
-		(property "Datasheet" "https://search.kemet.com/download/specsheet/C0603C473K5RACAUTO"
+		(property "Datasheet" "https://www.yageogroup.com/content/datasheet/asset/file/KEM_C1023_X7R_AUTO_SMD"
 			(at 0 0 270)
 			(layer "F.Fab")
@@
 			)
 		)
-		(property "Description" "0.047 µF ±10% 50V Ceramic Capacitor X7R 0603 (1608 Metric)"
+		(property "Description" "0.47 µF ±10% 25V Ceramic Capacitor X7R 0603 (1608 Metric)"
 			(at 0 0 270)
 			(layer "F.Fab")
@@
 			)
 		)
-		(property "DPN" "399-6820-1-ND"
+		(property "DPN" "399-C0603C474K3RACAUTOCT-ND"
 			(at 0 0 270)
 			(unlocked yes)
@@
 			)
 		)
-		(property "MPN" "C0603C473K5RACAUTO"
+		(property "MPN" "C0603C474K3RACAUTO"
 			(at 0 0 270)
 			(unlocked yes)
@@
 			)
 		)
-		(property "Value" "TCAN337G"
+		(property "Value" "TCAN337GDCN"
 			(at 0 2.4 90)
 			(layer "F.Fab")
@@
 			)
 		)
-		(property "Description" "1/1 Transceiver Half CANbus 8-SOIC"
+		(property "Description" "1/1 Transceiver Half CANbus SOT-23-8"
 			(at 0 0 90)
 			(layer "F.Fab")
@@
 			)
 		)
-		(property "DPN" "TCAN337GD-ND"
+		(property "DPN" "296-44539-1-ND"
 			(at 0 0 90)
 			(unlocked yes)
@@
 			)
 		)
-		(property "MPN" "TCAN337GD"
+		(property "MPN" "TCAN337GDCNT"
 			(at 0 0 90)
 			(unlocked yes)
@@
 			)
 		)
-		(property "Datasheet" "https://search.kemet.com/download/specsheet/C0603C473K5RACAUTO"
+		(property "Datasheet" "https://www.yageogroup.com/content/datasheet/asset/file/KEM_C1023_X7R_AUTO_SMD"
 			(at 0 0 180)
 			(layer "F.Fab")
@@
 			)
 		)
-		(property "Description" "0.047 µF ±10% 50V Ceramic Capacitor X7R 0603 (1608 Metric)"
+		(property "Description" "0.47 µF ±10% 25V Ceramic Capacitor X7R 0603 (1608 Metric)"
 			(at 0 0 180)
 			(layer "F.Fab")
@@
 			)
 		)
-		(property "DPN" "399-6820-1-ND"
+		(property "DPN" "399-C0603C474K3RACAUTOCT-ND"
 			(at 0 0 180)
 			(unlocked yes)
@@
 			)
 		)
-		(property "MPN" "C0603C473K5RACAUTO"
+		(property "MPN" "C0603C474K3RACAUTO"
 			(at 0 0 180)
 			(unlocked yes)
@@
 			)
 		)
-		(property "Datasheet" "https://search.kemet.com/download/specsheet/C0603C473K5RACAUTO"
+		(property "Datasheet" "https://www.yageogroup.com/content/datasheet/asset/file/KEM_C1023_X7R_AUTO_SMD"
 			(at 0 0 0)
 			(layer "F.Fab")
@@
 			)
 		)
-		(property "Description" "0.047 µF ±10% 50V Ceramic Capacitor X7R 0603 (1608 Metric)"
+		(property "Description" "0.47 µF ±10% 25V Ceramic Capacitor X7R 0603 (1608 Metric)"
 			(at 0 0 0)
 			(layer "F.Fab")
@@
 			)
 		)
-		(property "DPN" "399-6820-1-ND"
+		(property "DPN" "399-C0603C474K3RACAUTOCT-ND"
 			(at 0 0 0)
 			(unlocked yes)
@@
 			)
 		)
-		(property "MPN" "C0603C473K5RACAUTO"
+		(property "MPN" "C0603C474K3RACAUTO"
 			(at 0 0 0)
 			(unlocked yes)
@@
 			)
 		)
-		(property "Datasheet" "https://search.kemet.com/download/specsheet/C0603C473K5RACAUTO"
+		(property "Datasheet" "https://www.yageogroup.com/content/datasheet/asset/file/KEM_C1023_X7R_AUTO_SMD"
 			(at 0 0 180)
 			(layer "F.Fab")
@@
 			)
 		)
-		(property "Description" "0.047 µF ±10% 50V Ceramic Capacitor X7R 0603 (1608 Metric)"
+		(property "Description" "0.47 µF ±10% 25V Ceramic Capacitor X7R 0603 (1608 Metric)"
 			(at 0 0 180)
 			(layer "F.Fab")
@@
 			)
 		)
-		(property "DPN" "399-6820-1-ND"
+		(property "DPN" "399-C0603C474K3RACAUTOCT-ND"
 			(at 0 0 180)
 			(unlocked yes)
@@
 			)
 		)
-		(property "MPN" "C0603C473K5RACAUTO"
+		(property "MPN" "C0603C474K3RACAUTO"
 			(at 0 0 180)
 			(unlocked yes)
