File: oresat-battery-card/oresat-batteries-sch-pack-1.kicad_sch (KiCad schematic)
At the start: 92 parts, among them Q13 SI7111EDN-T1-GE3, Q14 DMP2035UQ-7, Q15 DMP2035UQ-7, Q16 SI7111EDN-T1-GE3, Q17 SI7111EDN-T1-GE3, Q18 SI7111EDN-T1-GE3, Q19 SI7111EDN-T1-GE3, Q23 DMP2035UQ-7, Q29 SQS484ENW-T1_GE3, Q6 DMN2053UQ-13, Q7 DMN2053UQ-13, Q8 DMN2053UQ-13, Q9 DMN2053UQ-13, U10 TPS259830ONRGER, U11 LTC4412, U12 MAX17205G, U8 S-8209AAA-T8T1U, U9 S-8209AAA-T8T1U

Commit message: Added imon capabilities, cleaned up some lingering DRCs that kept popping back up.
Parts:
- added C67: 100n, oresat-passives:0603-C-NOSILK, symbol Device:C_Small
- added R120: 10k, oresat-passives:0603-C-NOSILK, symbol Device:R_Small_US
Connections:
- net GND: now also C67.2
- net at R72.1, TP37.1, U10.9 (IMON): now also R120.1
- new net IMON-PK1: C67.1, R120.2

Commit message: Changes after inventory check and BOM check
Parts:
- C24, C25: DPN 399-6820-1-ND -> 399-C0603C474K3RACAUTOCT-ND; MPN C0603C473K5RACAUTO -> C0603C474K3RACAUTO
Changed lines of the file:
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@@
 			)
 		)
-		(property "Datasheet" "https://search.kemet.com/download/specsheet/C0603C473K5RACAUTO"
+		(property "Datasheet" "https://www.yageogroup.com/content/datasheet/asset/file/KEM_C1023_X7R_AUTO_SMD"
 			(at 474.98 189.23 0)
 			(hide yes)
@@
 			)
 		)
-		(property "Description" "0.047 µF ±10% 50V Ceramic Capacitor X7R 0603 (1608 Metric)"
+		(property "Description" "0.47 µF ±10% 25V Ceramic Capacitor X7R 0603 (1608 Metric)"
 			(at 474.98 189.23 0)
 			(hide yes)
@@
 			)
 		)
-		(property "DPN" "399-6820-1-ND"
+		(property "DPN" "399-C0603C474K3RACAUTOCT-ND"
 			(at 474.98 189.23 0)
 			(hide yes)
@@
 			)
 		)
-		(property "MPN" "C0603C473K5RACAUTO"
+		(property "MPN" "C0603C474K3RACAUTO"
 			(at 474.98 189.23 0)
 			(hide yes)
@@
 			)
 		)
-		(property "Datasheet" "https://search.kemet.com/download/specsheet/C0603C473K5RACAUTO"
+		(property "Datasheet" "https://www.yageogroup.com/content/datasheet/asset/file/KEM_C1023_X7R_AUTO_SMD"
 			(at 485.14 189.23 0)
 			(hide yes)
@@
 			)
 		)
-		(property "Description" "0.047 µF ±10% 50V Ceramic Capacitor X7R 0603 (1608 Metric)"
+		(property "Description" "0.47 µF ±10% 25V Ceramic Capacitor X7R 0603 (1608 Metric)"
 			(at 485.14 189.23 0)
 			(hide yes)
@@
 			)
 		)
-		(property "DPN" "399-6820-1-ND"
+		(property "DPN" "399-C0603C474K3RACAUTOCT-ND"
 			(at 485.14 189.23 0)
 			(hide yes)
@@
 			)
 		)
-		(property "MPN" "C0603C473K5RACAUTO"
+		(property "MPN" "C0603C474K3RACAUTO"
 			(at 485.14 189.23 0)
 			(hide yes)
